Commit message: Modify original model files

File: urdf/base_original.xacro (robot description, xacro)
@@ -17,5 +17,5 @@
             <inertial>
                 <origin rpy="0 0 0" xyz="0 0 0"/>
-                <mass value="819026.342183402"/>
+                <mass value="819026"/>
                 <!--<inertia ixx="1439809.19440102" ixy="205163.256495052" ixz="-240460.141925145" iyy="24924095.2244092" iyz="-3294.60477684522" izz="25510047.9278752"/>-->
                 <inertia ixx="1439809.19440102" ixy="0.0" ixz="0.0" iyy="24924095.2244092" iyz="0.0" izz="25510047.9278752"/>

File: urdf/gazebo_original.xacro (robot description, xacro)
@@ -135,10 +135,10 @@
           </added_mass>
           <!--<added_mass>
-            1.432   0       0       0     0      0
-            0    120.645    0       0     0    4.895
-            0       0    130.513    0  -16.488   0
-            0       0       0    0.386    0      0
-            0       0   -16.488     0  78.266    0
-            0     4.895     0       0     0    67.489
+              1.432   0       0       0     0      0
+              0    120.645    0       0     0    4.895
+              0       0    130.513    0  -16.488   0
+              0       0       0    0.386    0      0
+              0       0   -16.488     0  78.266    0
+              0     4.895     0       0     0    67.489
           </added_mass>-->
           <!--
@@ -176,10 +176,10 @@
           </quadratic_damping>
           <!--<quadratic_damping>
-            -3.9     0      0      0     0      0
-              0  -373.287   0      0     0   -4.204
-              0      0  -489.07    0  23.016    0
-              0      0      0   -0.117   0      0
-              0      0   23.342    0 -353.406   0
-              0   0.419     0      0     0  -227.024
+              -3.9     0      0      0     0      0
+                0  -373.287   0      0     0   -4.204
+                0      0  -489.07    0  23.016    0
+                0      0      0   -0.117   0      0
+                0      0   23.342    0 -353.406   0
+                0   0.419     0      0     0  -227.024
           </quadratic_damping>-->
         </hydrodynamic_model>

File: urdf/snippets_original.xacro (robot description, xacro)
@@ -92,6 +92,8 @@
   <xacro:property name="fin_rho" value="1025"/>
   <xacro:property name="front_fin_area" value="2.9153726"/>
-  <xacro:property name="front_fin_lift_coefficient" value="1.668475641"/>
-  <xacro:property name="front_fin_drag_coefficient" value="0.26542681"/>
+  <!--<xacro:property name="front_fin_lift_coefficient" value="1.668475641"/>-->
+  <xacro:property name="front_fin_lift_coefficient" value="20.843"/>
+  <!--<xacro:property name="front_fin_drag_coefficient" value="0.26542681"/>-->
+  <xacro:property name="front_fin_drag_coefficient" value="1.98"/>
   <xacro:macro name="front_left_fin_macro" params="namespace fin_id *origin mesh_filename">
     <xacro:hor_left_fin_quadratic_macro
@@ -204,6 +206,8 @@
   <xacro:property name="aft_fin_area" value="2.656049"/>
   <!--<xacro:property name="aft_fin_area" value="0.785"/>-->
-  <xacro:property name="aft_fin_lift_coefficient" value="1.74975211"/>
-  <xacro:property name="aft_fin_drag_coefficient" value="0.269448395"/>
+  <!--<xacro:property name="aft_fin_lift_coefficient" value="1.74975211"/>-->
+  <xacro:property name="aft_fin_lift_coefficient" value="19.1395"/>
+  <!--<xacro:property name="aft_fin_drag_coefficient" value="0.269448395"/>-->
+  <xacro:property name="aft_fin_drag_coefficient" value="1.98"/>
   <xacro:macro name="back_up_fin_macro" params="namespace fin_id *origin mesh_filename">
     <xacro:lat_up_fin_quadratic_macro
