Commit message: Try original parameters of hydrodynamic

File: urdf/gazebo.xacro (robot description, xacro)
@@ -6,4 +6,5 @@
     <!--<xacro:property name="O_29qt_volume" value="${819026 / 9.8 / 1000}"/>-->
     <xacro:property name="O_29qt_volume" value="${838 / 9.8 / 1000}"/>
+    <!--<xacro:property name="O_29qt_volume" value="${4690 / 1000}"/>-->
     <!-- Describing the dimensions of the vehicle's bounding box -->
     <!--<xacro:property name="O_29qt_length" value="40.97"/>
@@ -11,8 +12,14 @@
     <xacro:property name="O_29qt_radius"  value="2.4615"/>
     <xacro:property name="O_29qt_height" value="4.923"/>-->
+    <!-- Added base parameters(ARMSAUA) -->
     <xacro:property name="O_29qt_length" value="2.712"/>
     <xacro:property name="O_29qt_width"  value="0.935"/>
     <xacro:property name="O_29qt_radius"  value="0.120"/>
     <xacro:property name="O_29qt_height" value="0.484"/>
+    <!-- Added base parameters -->
+    <!--<xacro:property name="O_29qt_length" value="8.534"/>
+    <xacro:property name="O_29qt_width"  value="2.94525"/>
+    <xacro:property name="O_29qt_radius"  value="0.5128"/>
+    <xacro:property name="O_29qt_height" value="1.5246"/>-->
     <xacro:property name="rho" value="1025" />
     <xacro:property name="D0" value="${rho * 0.5}"/>
@@ -24,4 +31,78 @@
     <xacro:property name="D00" value="0.7159"/>
     <xacro:property name="D04" value="0.2627"/>
+    <xacro:property name="xudot" value="-0.000949"/>
+    <xacro:property name="xvdot" value="0.0"/>
+    <xacro:property name="xwdot" value="0.0"/>
+    <xacro:property name="xpdot" value="0.0"/>
+    <xacro:property name="xqdot" value="0.0"/>
+    <xacro:property name="xrdot" value="0.0"/>
+    <xacro:property name="yudot" value="0.0"/>
+    <xacro:property name="yvdot" value="-0.0408"/>
+    <xacro:property name="ywdot" value="0.0"/>
+    <xacro:property name="ypdot" value="0.000547"/>
+    <xacro:property name="yqdot" value="0.0"/>
+    <xacro:property name="yrdot" value="0.00139"/>
+    <xacro:property name="zudot" value="0.0"/>
+    <xacro:property name="zvdot" value="0.0"/>
+    <xacro:property name="zwdot" value="-0.0226"/>
+    <xacro:property name="zpdot" value="0.0"/>
+    <xacro:property name="zqdot" value="-0.0000510"/>
+    <xacro:property name="zrdot" value="0.0"/>
+    <xacro:property name="kudot" value="0.0"/>
+    <xacro:property name="kvdot" value="0.000547"/>
+    <xacro:property name="kwdot" value="0.0"/>
+    <xacro:property name="kpdot" value="-0.000105"/>
+    <xacro:property name="kqdot" value="0.0"/>
+    <xacro:property name="krdot" value="-0.00000370"/>
+    <xacro:property name="mudot" value="0.0"/>
+    <xacro:property name="mvdot" value="0.0"/>
+    <xacro:property name="mwdot" value="-0.0000510"/>
+    <xacro:property name="mpdot" value="0.0"/>
+    <xacro:property name="mqdot" value="-0.00175"/>
+    <xacro:property name="mrdot" value="0.0"/>
+    <xacro:property name="nudot" value="0.0"/>
+    <xacro:property name="nvdot" value="0.00139"/>
+    <xacro:property name="nwdot" value="0.0"/>
+    <xacro:property name="npdot" value="-0.00000370"/>
+    <xacro:property name="nqdot" value="0.0"/>
+    <xacro:property name="nrdot" value="-0.00183"/>
+    <!-- Damping -->
+    <xacro:property name="xuu" value="-0.00315"/>
+    <xacro:property name="xuv" value="0.0"/>
+    <xacro:property name="xuw" value="0.0"/>
+    <xacro:property name="xup" value="0.0"/>
+    <xacro:property name="xuq" value="0.0"/>
+    <xacro:property name="xur" value="0.0"/>
+    <xacro:property name="yuu" value="0.0"/>
+    <xacro:property name="yuv" value="-0.099"/>
+    <xacro:property name="yuw" value="0.0"/>
+    <xacro:property name="yup" value="0.00677"/>
+    <xacro:property name="yuq" value="0.0"/>
+    <xacro:property name="yur" value="0.0250"/>
+    <xacro:property name="zuu" value="0.0"/>
+    <xacro:property name="zuv" value="0.0"/>
+    <xacro:property name="zuw" value="-0.067"/>
+    <xacro:property name="zup" value="0.0"/>
+    <xacro:property name="zuq" value="-0.00658"/>
+    <xacro:property name="zur" value="0.0"/>
+    <xacro:property name="kuu" value="0.0"/>
+    <xacro:property name="kuv" value="0.00406"/>
+    <xacro:property name="kuw" value="0.0"/>
+    <xacro:property name="kup" value="-0.00145"/>
+    <xacro:property name="kuq" value="0.0"/>
+    <xacro:property name="kur" value="-0.000578"/>
+    <xacro:property name="muu" value="0.0"/>
+    <xacro:property name="muv" value="0.0"/>
+    <xacro:property name="muw" value="0.00120"/>
+    <xacro:property name="mup" value="0.0"/>
+    <xacro:property name="muq" value="-0.00687"/>
+    <xacro:property name="mur" value="0.0"/>
+    <xacro:property name="nuu" value="0.0"/>
+    <xacro:property name="nuv" value="-0.005"/>
+    <xacro:property name="nuw" value="0.0"/>
+    <xacro:property name="nup" value="0.000086"/>
+    <xacro:property name="nuq" value="0.0"/>
+    <xacro:property name="nur" value="-0.00747"/>
+    <!-- Model setting -->
     <xacro:macro name="O_29qt_hydro_model" params="namespace">
       <!-- List of hydrodynamic models this robot's links -->
@@ -44,11 +125,11 @@
         <hydrodynamic_model>
           <type>fossen</type>
-          <!-- <added_mass>
-            ${-0.000949*D3*0.1}         0                 0                  0                   0                  0
-                      0         ${-0.0408*D3*0.1}         0         ${0.000547*D4*0.1}           0          ${0.00139*D4*0.1}
-                      0                 0         ${-0.0226*D3*0.1}          0         ${-0.0000510*D4*0.1}         0
-                      0         ${0.000547*D4*0.1}        0         ${-0.000105*D5*0.1}          0          ${-0.00000370*D5*0.1}
-                      0                 0         ${-0.0000510*D4*0.1}       0         ${-0.00175*D5*0.1}           0
-                      0         ${0.00139*D4*0.1}         0         ${-0.00000370*D5*0.1}        0          ${-0.00183*D5*0.1}
+          <!--<added_mass>
+              ${-xudot*D3*0.1}      ${-xvdot*D3*0.1}       ${-xwdot*D3*0.1}       ${-xpdot*D4*0.1}      ${-xqdot*D4*0.1}      ${-xrdot*D4*0.1}
+              ${-yudot*D3*0.1}      ${-yvdot*D3*0.1}       ${-ywdot*D3*0.1}       ${-ypdot*D4*0.1}      ${-yqdot*D4*0.1}      ${-yrdot*D4*0.1}
+              ${-zudot*D3*0.1}      ${-zvdot*D3*0.1}       ${-zwdot*D3*0.1}       ${-zpdot*D4*0.1}      ${-zqdot*D4*0.1}      ${-zrdot*D4*0.1}
+              ${-kudot*D4*0.1}      ${-kvdot*D4*0.1}       ${-kwdot*D4*0.1}       ${-kpdot*D5*0.1}      ${-kqdot*D5*0.1}      ${-krdot*D5*0.1}
+              ${-mudot*D4*0.1}      ${-mvdot*D4*0.1}       ${-mwdot*D4*0.1}       ${-mpdot*D5*0.1}      ${-mqdot*D5*0.1}      ${-mrdot*D5*0.1}
+              ${-nudot*D4*0.1}      ${-nvdot*D4*0.1}       ${-nwdot*D4*0.1}       ${-npdot*D5*0.1}      ${-nqdot*D5*0.1}      ${-nrdot*D5*0.1}
           </added_mass>-->
           <added_mass>
@@ -86,10 +167,10 @@
           -->
           <!--<quadratic_damping>
-            ${-0.00315*D2}       0           0             0             0             0
-                   0       ${-0.099*D2}      0       ${0.00677*D3}       0       ${0.0250*D3}
-                   0             0      ${-0.067*D2}       0      ${-0.00658*D3}       0
-                   0       ${0.00406*D3}     0       ${-0.00145*D4}      0      ${-0.000578*D4}
-                   0             0      ${0.00120*D3}      0      ${-0.00687*D4}       0
-                   0       ${-0.005*D3}      0       ${0.000086*D4}      0       ${-0.00747*D4}
+              ${xuu*D2}      ${xuv*D2}       ${xuw*D2}       ${xup*D3}      ${xuq*D3}      ${xur*D3}
+              ${yuu*D2}      ${yuv*D2}       ${yuw*D2}       ${yup*D3}      ${yuq*D3}      ${yur*D3}
+              ${zuu*D2}      ${zuv*D2}       ${zuw*D2}       ${zup*D3}      ${zuq*D3}      ${zur*D3}
+              ${kuu*D3}      ${kuv*D3}       ${kuw*D3}       ${kup*D4}      ${kuq*D4}      ${kur*D4}
+              ${muu*D3}      ${muv*D3}       ${muw*D3}       ${mup*D4}      ${muq*D4}      ${mur*D4}
+              ${nuu*D3}      ${nuv*D3}       ${nuw*D3}       ${nup*D4}      ${nuq*D4}      ${nur*D4}
           </quadratic_damping>-->
           <quadratic_damping>

Commit message: restore default parameters

File: urdf/gazebo.xacro (robot description, xacro)
@@ -5,6 +5,6 @@
     <!-- Vehicle's actual volume (Gazebo cannot compute the volume out of the mesh) -->
     <!--<xacro:property name="O_29qt_volume" value="${819026 / 9.8 / 1000}"/>-->
-    <xacro:property name="O_29qt_volume" value="${838 / 9.8 / 1000}"/>
-    <!--<xacro:property name="O_29qt_volume" value="${4690 / 1000}"/>-->
+    <!--<xacro:property name="O_29qt_volume" value="${838 / 9.8 / 1000}"/>-->
+    <xacro:property name="O_29qt_volume" value="${4690 / 1000}"/>
     <!-- Describing the dimensions of the vehicle's bounding box -->
     <!--<xacro:property name="O_29qt_length" value="40.97"/>
@@ -13,13 +13,13 @@
     <xacro:property name="O_29qt_height" value="4.923"/>-->
     <!-- Added base parameters(ARMSAUA) -->
-    <xacro:property name="O_29qt_length" value="2.712"/>
+    <!--<xacro:property name="O_29qt_length" value="2.712"/>
     <xacro:property name="O_29qt_width"  value="0.935"/>
     <xacro:property name="O_29qt_radius"  value="0.120"/>
-    <xacro:property name="O_29qt_height" value="0.484"/>
+    <xacro:property name="O_29qt_height" value="0.484"/>-->
     <!-- Added base parameters -->
-    <!--<xacro:property name="O_29qt_length" value="8.534"/>
+    <xacro:property name="O_29qt_length" value="8.534"/>
     <xacro:property name="O_29qt_width"  value="2.94525"/>
     <xacro:property name="O_29qt_radius"  value="0.5128"/>
-    <xacro:property name="O_29qt_height" value="1.5246"/>-->
+    <xacro:property name="O_29qt_height" value="1.5246"/>
     <xacro:property name="rho" value="1025" />
     <xacro:property name="D0" value="${rho * 0.5}"/>
@@ -125,5 +125,5 @@
         <hydrodynamic_model>
           <type>fossen</type>
-          <!--<added_mass>
+          <added_mass>
               ${-xudot*D3*0.1}      ${-xvdot*D3*0.1}       ${-xwdot*D3*0.1}       ${-xpdot*D4*0.1}      ${-xqdot*D4*0.1}      ${-xrdot*D4*0.1}
               ${-yudot*D3*0.1}      ${-yvdot*D3*0.1}       ${-ywdot*D3*0.1}       ${-ypdot*D4*0.1}      ${-yqdot*D4*0.1}      ${-yrdot*D4*0.1}
@@ -132,6 +132,6 @@
               ${-mudot*D4*0.1}      ${-mvdot*D4*0.1}       ${-mwdot*D4*0.1}       ${-mpdot*D5*0.1}      ${-mqdot*D5*0.1}      ${-mrdot*D5*0.1}
               ${-nudot*D4*0.1}      ${-nvdot*D4*0.1}       ${-nwdot*D4*0.1}       ${-npdot*D5*0.1}      ${-nqdot*D5*0.1}      ${-nrdot*D5*0.1}
-          </added_mass>-->
-          <added_mass>
+          </added_mass>
+          <!--<added_mass>
             1.432   0       0       0     0      0
             0    120.645    0       0     0    4.895
@@ -140,5 +140,5 @@
             0       0   -16.488     0  78.266    0
             0     4.895     0       0     0    67.489
-          </added_mass>
+          </added_mass>-->
           <!--
             The linear damping coefficients can be provided as a diagonal (6 elements)
@@ -166,5 +166,5 @@
             or a full matrix (36 coefficients), like the added-mass coefficients above
           -->
-          <!--<quadratic_damping>
+          <quadratic_damping>
               ${xuu*D2}      ${xuv*D2}       ${xuw*D2}       ${xup*D3}      ${xuq*D3}      ${xur*D3}
               ${yuu*D2}      ${yuv*D2}       ${yuw*D2}       ${yup*D3}      ${yuq*D3}      ${yur*D3}
@@ -173,6 +173,6 @@
               ${muu*D3}      ${muv*D3}       ${muw*D3}       ${mup*D4}      ${muq*D4}      ${mur*D4}
               ${nuu*D3}      ${nuv*D3}       ${nuw*D3}       ${nup*D4}      ${nuq*D4}      ${nur*D4}
-          </quadratic_damping>-->
-          <quadratic_damping>
+          </quadratic_damping>
+          <!--<quadratic_damping>
             -3.9     0      0      0     0      0
               0  -373.287   0      0     0   -4.204
@@ -181,5 +181,5 @@
               0      0   23.342    0 -353.406   0
               0   0.419     0      0     0  -227.024
-          </quadratic_damping>
+          </quadratic_damping>-->
         </hydrodynamic_model>
       </link>

File: urdf/snippets.xacro (robot description, xacro)
@@ -39,7 +39,7 @@
                 <clampMin>-2300</clampMin>
                 <!-- Maximum thrust force output allowed -->
-                <thrustMax>1250</thrustMax>
+                <thrustMax>26338.811</thrustMax>
                 <!-- Minimum thrust force output allowed -->
-                <thrustMin>-1250</thrustMin>
+                <thrustMin>-26338.811</thrustMin>
                 <!--
                 Value from 0 to 1 to set the efficiency of the output thrus

Commit message: Test small size model

File: urdf/gazebo.xacro (robot description, xacro)
@@ -77,6 +77,5 @@
     <xacro:property name="kuu" value="0.0"/>
     <xacro:property name="kuv" value="0.00406"/>
-    <xacro:property name="kuw" value="0.0"/>
-    <xacro:property name="kup" value="-0.00145"/>
+    <xacro:property name="kuw" value="0.0"/> <xacro:property name="kup" value="-0.00145"/>
     <xacro:property name="kuq" value="0.0"/>
     <xacro:property name="kur" value="-0.000578"/>

File: urdf/snippets.xacro (robot description, xacro)
@@ -1,5 +1,5 @@
 <?xml version="1.0" encoding="UTF-8"?>
 <robot xmlns:xacro="http://www.ros.org/wiki/xacro">
-    <xacro:property name="propeller_mesh_file" value="file://$(find O_29qt)/meshes/propeller.STL" />
+    <xacro:property name="propeller_mesh_file" value="file://$(find armsauv_description)/meshes/propeller.dae" />
     <xacro:macro name="thruster_macro" params="robot_namespace thruster_id *origin">
         <link name="${robot_namespace}/thruster_${thruster_id}">
@@ -85,18 +85,14 @@
     <!-- MACRO FOR FIN/RUDDER UNITS  -->
   <!-- A separate mesh for the fin should be stored in the meshes folder -->
-  <xacro:property name="front_fin_mesh_file" value="file://$(find O_29qt)/meshes/front_fin_latest.STL"/>
-  <!--<xacro:property name="front_fin_mesh_file" value="file://$(find armsauv_description)/meshes/front_fin.dae"/>-->
-  <xacro:property name="aft_fin_mesh_file" value="file://$(find O_29qt)/meshes/aft_fin_latest.STL"/>
-  <!--<xacro:property name="aft_fin_mesh_file" value="file://$(find armsauv_description)/meshes/aft_fin.dae"/>-->
+  <xacro:property name="front_fin_mesh_file" value="file://$(find armsauv_description)/meshes/front_fin.dae"/>
+  <xacro:property name="aft_fin_mesh_file" value="file://$(find armsauv_description)/meshes/aft_fin.dae"/>
   <!-- Fin properties -->
   <xacro:property name="fin_rho" value="1025"/>
-  <!--<xacro:property name="front_fin_area" value="2.9153726"/>-->
   <!--<xacro:property name="front_fin_area" value="0.0127"/>-->
   <xacro:property name="front_fin_area" value="0.116615"/>
-  <!--<xacro:property name="front_fin_lift_coefficient" value="1.668475641"/>-->
   <xacro:property name="front_fin_lift_coefficient" value="3.416017484"/>
   <xacro:property name="front_fin_drag_coefficient" value="0.26542681"/>
   <xacro:macro name="front_fin_macro" params="namespace fin_id *origin mesh_filename">
-      <!--<xacro:fin_quadratic_macro
+      <xacro:fin_quadratic_macro
         namespace="${namespace}"
         parent_link="${namespace}/base_link" fin_id="${fin_id}"
@@ -110,46 +106,11 @@
         <xacro:insert_block name="origin"/>
       </xacro:fin_quadratic_macro>-->
-      <link name="${namespace}/fin${fin_id}">
-          <xacro:no_inertial/>
-          <visual>
-              <origin xyz="0 0 0" rpy="0 0 0"/>
-              <geometry>
-                  <mesh filename="${mesh_filename}" scale="1 1 1"/>
-              </geometry>
-          </visual>
-      </link>
-      <joint name="${namespace}/fin${fin_id}_joint" type="revolute">
-          <limit effort="0" lower="${-90*d2r}" upper="${90*d2r}" velocity="0"/>
-          <xacro:insert_block name="origin"/>
-          <axiz xyz="0 0 1"/>
-          <parent link="${namespace}/base_link"/>
-          <child link="${namespace}/fin${fin_id}"/>
-      </joint>
-      <gazebo>
-          <plugin name="${namespace}_fin${fin_id}_model" filename="libuuv_fin_ros_plugin.so">
-              <dynamics>
-                  <type>FirstOrder</type>
-                  <timeConstant>0.2</timeConstant>
-              </dynamics>
-              <liftdrag>
-                  <type>Quadratic</type>
-                  <lift_constant>${0.5 * fin_rho * front_fin_area * front_fin_lift_coefficient}</lift_constant>
-                  <drag_constant>${0.5 * fin_rho * front_fin_area * front_fin_drag_coefficient}</drag_constant>
-              </liftdrag>
-              <current_velocity_topic>current_velocity</current_velocity_topic>
-              <fin_id>${fin_id}</fin_id>
-              <link_name>${namespace}/fin${fin_id}</link_name>
-              <joint_name>${namespace}/fin${fin_id}_joint</joint_name>
-          </plugin>
-      </gazebo>
   </xacro:macro>
-  <!--<xacro:property name="aft_fin_area" value="2.656049"/>-->
   <!--<xacro:property name="aft_fin_area" value="0.0172"/>-->
   <xacro:property name="aft_fin_area" value="0.106243"/>
-  <!--<xacro:property name="aft_fin_lift_coefficient" value="1.74975211"/>-->
   <xacro:property name="aft_fin_lift_coefficient" value="3.290443227"/>
   <xacro:property name="aft_fin_drag_coefficient" value="0.269448395"/>
   <xacro:macro name="aft_fin_macro" params="namespace fin_id *origin mesh_filename">
-      <!--<xacro:fin_quadratic_macro
+      <xacro:fin_quadratic_macro
         namespace="${namespace}"
         parent_link="${namespace}/base_link"
@@ -163,82 +124,5 @@
         current_velocity_topic="current_velocity">
         <xacro:insert_block name="origin"/>
-      </xacro:fin_quadratic_macro>-->
-      <link name="${namespace}/fin${fin_id}">
-          <xacro:no_inertial/>
-          <visual>
-              <origin xyz="0 0 0" rpy="0 0 0"/>
-              <geometry>
-                  <mesh filename="${mesh_filename}" scale="1 1 1"/>
-              </geometry>
-          </visual>
-      </link>
-      <joint name="${namespace}/fin${fin_id}_joint" type="revolute">
-          <limit effort="0" lower="${-90*d2r}" upper="${90*d2r}" velocity="0"/>
-          <xacro:insert_block name="origin"/>
-          <axiz xyz="0 0 1"/>
-          <parent link="${namespace}/base_link"/>
-          <child link="${namespace}/fin${fin_id}"/>
-      </joint>
-      <gazebo>
-          <plugin name="${namespace}_fin${fin_id}_model" filename="libuuv_fin_ros_plugin.so">
-              <dynamics>
-                  <type>FirstOrder</type>
-                  <timeConstant>0.2</timeConstant>
-              </dynamics>
-              <liftdrag>
-                  <type>Quadratic</type>
-                  <lift_constant>${0.5 * fin_rho * front_fin_area * front_fin_lift_coefficient}</lift_constant>
-                  <drag_constant>${0.5 * fin_rho * front_fin_area * front_fin_drag_coefficient}</drag_constant>
-              </liftdrag>
-              <current_velocity_topic>current_velocity</current_velocity_topic>
-              <fin_id>${fin_id}</fin_id>
-              <link_name>${namespace}/fin${fin_id}</link_name>
-              <joint_name>${namespace}/fin${fin_id}_joint</joint_name>
-          </plugin>
-      </gazebo>
+      </xacro:fin_quadratic_macro>
   </xacro:macro>
-  <!-- <xacro:macro name="fin_macro" params="namespace fin_id *origin mesh_filename">
-      <xacro:fin_two_lines_macro
-        namespace="${namespace}"
-        parent_link="${namespace}/base_link"
-        fin_id="${fin_id}"
-        min_joint_limit="${-80*d2r}"
-        max_joint_limit="${80*d2r}"
-        mesh_filename="${mesh_filename}"
-        fin_dynamics_time_constant="0.1"
-        fin_cross_section_area="${fin_area}"
-        current_velocity_topic="current_velocity"
-        fluid_density="1025.0"
-        a0="0.0"
-        alpha_stall="1.57"
-        cla="${0.5 * fin_rho * fin_area * fin_lift_coefficient}"
-        cla_stall="0.0"
-        cda="${0.5 * fin_rho * fin_area * fin_drag_coefficient}"
-        cda_stall="0">
-        <xacro:insert_block name="origin"/>
-      </xacro:fin_two_lines_macro>
-    </xacro:macro> -->
-    <!-- <xacro:macro name="fin_macro" params="namespace fin_id *origin mesh_filename">
-      <xacro:fin_two_lines_macro
-        namespace="${namespace}"
-        parent_link="${namespace}/base_link"
-        fin_id="${fin_id}"
-        min_joint_limit="${-80*d2r}"
-        max_joint_limit="${80*d2r}"
-        mesh_filename="${mesh_filename}"
-        fin_dynamics_time_constant="0.1"
-        fin_cross_section_area="${fin_area}"
-        current_velocity_topic="current_velocity"
-        fluid_density="1025.0"
-        a0="0.0"
-        alpha_stall="0.436332313"
-        cla="2.435070629"
-        cla_stall="0"
-        cda="0"
-        cda_stall="0">
-        <xacro:insert_block name="origin"/>
-      </xacro:fin_two_lines_macro>
-    </xacro:macro> -->
-    <!-- cla_stall="-1.929963096"
-        cda="1.101841914" -->
 </robot>
