Commit message: Remove redundant sensors for O29 model

File: urdf/sensors_original.xacro (robot description, xacro)
@@ -62,9 +62,9 @@
     </xacro:Imu>
     <!-- DVL  -->
-    <xacro:default_dvl namespace="${namespace}" parent_link="${namespace}/base_link">
+    <!--<xacro:default_dvl namespace="${namespace}" parent_link="${namespace}/base_link">
       <origin xyz="0 0 0" rpy="0 0 0"/>
-    </xacro:default_dvl>
+    </xacro:default_dvl>-->
     <!-- Mount a Pressure Sensor -->
-    <xacro:macro name="Pressure" params="namespace parent_link *origin">
+    <!--<xacro:macro name="Pressure" params="namespace parent_link *origin">
       <xacro:pressure_plugin_macro
         namespace="${namespace}"
@@ -83,7 +83,7 @@
         <origin xyz="0 0 0" rpy="0 0 0"/>
       </xacro:pressure_plugin_macro>
-    </xacro:macro>
-    <xacro:Pressure namespace="${namespace}" parent_link="${namespace}/base_link">
+    </xacro:macro>-->
+    <!--<xacro:Pressure namespace="${namespace}" parent_link="${namespace}/base_link">
         <origin xyz="0 0 0" rpy="0 0 0"/>
-    </xacro:Pressure>
+    </xacro:Pressure>-->
 </robot>
