Commit message: Try original parameters of actuators

File: urdf/actuators.xacro (robot description, xacro)
@@ -8,24 +8,30 @@
         <!--<origin xyz="10.2108 -2.3958 -1.3989" rpy="${0.5 * pi} 0 0" />-->
         <origin xyz="0.528 -0.201 0" rpy="${0.5 * pi} 0 0" />
+        <!--<origin xyz="1.6632 -0.63315 0" rpy="${0.5 * pi} 0 0" />-->
     </xacro:front_fin_macro>
     <xacro:front_fin_macro namespace="${namespace}" fin_id="1" mesh_filename="${front_fin_mesh_file}">
         <!--<origin xyz="10.2108 2.3958 -1.3989" rpy="${1.5 * pi} 0 0" />-->
         <origin xyz="0.528 0.201 0" rpy="${1.5 * pi} 0 0" />
+        <!--<origin xyz="1.6632 0.63315 0" rpy="${1.5 * pi} 0 0" />-->
     </xacro:front_fin_macro>
     <xacro:aft_fin_macro namespace="${namespace}" fin_id="2" mesh_filename="${aft_fin_mesh_file}">
         <!--<origin xyz="-16.583 2.2397 -0.4013" rpy="${0.5 * pi} 0 0" />-->
         <origin xyz="-1.537 0.136 0" rpy="${0.5 * pi} 0 0" />
+        <!--<origin xyz="-4.84155 0.4284 0" rpy="${0.5 * pi} 0 0" />-->
     </xacro:aft_fin_macro>
     <xacro:aft_fin_macro namespace="${namespace}" fin_id="3" mesh_filename="${aft_fin_mesh_file}">
         <!--<origin xyz="-16.583 0.0 2.25677" rpy="${1.0 * pi} 0 0" />-->
         <origin xyz="-1.537 0 0.136" rpy="${1.0 * pi} 0 0" />
+        <!--<origin xyz="-4.84155 0 0.4284" rpy="${1.0 * pi} 0 0" />-->
     </xacro:aft_fin_macro>
     <xacro:aft_fin_macro namespace="${namespace}" fin_id="4" mesh_filename="${aft_fin_mesh_file}">
         <!--<origin xyz="-16.583 -2.2397 -0.4013" rpy="${1.5 * pi} 0 0" />-->
         <origin xyz="-1.537 -0.136 0" rpy="${1.5 * pi} 0 0" />
+        <!--<origin xyz="-4.84155 -0.4284 0" rpy="${1.5 * pi} 0 0" />-->
     </xacro:aft_fin_macro>
     <xacro:aft_fin_macro namespace="${namespace}" fin_id="5" mesh_filename="${aft_fin_mesh_file}">
         <!--<origin xyz="-16.583 0.0 -2.25677" rpy="${0.0 * pi} 0 0" />-->
         <origin xyz="-1.537 0 -0.136" rpy="${0.0 * pi} 0 0" />
+        <!--<origin xyz="-4.84155 0 -0.4284" rpy="${0.0 * pi} 0 0" />-->
     </xacro:aft_fin_macro>
 </robot>

Commit message: Test lift and drag coefficient of fins

File: urdf/actuators.xacro (robot description, xacro)
@@ -2,36 +2,33 @@
 <robot xmlns:xacro="http://www.ros.org/wiki/xacro">
     <xacro:thruster_macro robot_namespace="${namespace}" thruster_id = "0">
-        <!--<origin xyz="-20.432 0.0 0.1958" rpy="0 0 0" />-->
-        <origin xyz="-1.842 0.0 0" rpy="0 0 0" />
+        <origin xyz="-4.668392 0.0 0" rpy="0 0 0" />
     </xacro:thruster_macro>
     <xacro:front_fin_macro namespace="${namespace}" fin_id="0" mesh_filename="${front_fin_mesh_file}">
-        <!--<origin xyz="10.2108 -2.3958 -1.3989" rpy="${0.5 * pi} 0 0" />-->
-        <origin xyz="0.528 -0.201 0" rpy="${0.5 * pi} 0 0" />
-        <!--<origin xyz="1.6632 -0.63315 0" rpy="${0.5 * pi} 0 0" />-->
+        <!--<origin xyz="2.168598 0.4569450 0.27093419" rpy="0 0 0" />-->
+        <!--<origin xyz="2.168598 -0.4569450 0.27093419" rpy="${0.5 * pi} 0 0" />-->
+        <origin xyz="2.168598 -0.4569450 0.0" rpy="${0.5 * pi} 0 0" />
     </xacro:front_fin_macro>
     <xacro:front_fin_macro namespace="${namespace}" fin_id="1" mesh_filename="${front_fin_mesh_file}">
-        <!--<origin xyz="10.2108 2.3958 -1.3989" rpy="${1.5 * pi} 0 0" />-->
-        <origin xyz="0.528 0.201 0" rpy="${1.5 * pi} 0 0" />
-        <!--<origin xyz="1.6632 0.63315 0" rpy="${1.5 * pi} 0 0" />-->
+        <!--<origin xyz="2.168598 -0.4569450 0.27093419" rpy="${1.0 * pi} 0 0" />-->
+        <!--<origin xyz="2.168598 0.4569450 0.27093419" rpy="${1.5 * pi} 0 0" />-->
+        <origin xyz="2.168598 0.4569450 0.0" rpy="${1.5 * pi} 0 0" />
     </xacro:front_fin_macro>
     <xacro:aft_fin_macro namespace="${namespace}" fin_id="2" mesh_filename="${aft_fin_mesh_file}">
-        <!--<origin xyz="-16.583 2.2397 -0.4013" rpy="${0.5 * pi} 0 0" />-->
-        <origin xyz="-1.537 0.136 0" rpy="${0.5 * pi} 0 0" />
-        <!--<origin xyz="-4.84155 0.4284 0" rpy="${0.5 * pi} 0 0" />-->
+        <!--<origin xyz="-3.4129751 0.46646423 0.05598445" rpy="0 0 0" />-->
+        <!--<origin xyz="-3.4129751 0.46646423 0.05598445" rpy="${0.5 * pi} 0 0" />-->
+        <origin xyz="-3.4129751 0.46646423 0.0" rpy="${0.5 * pi} 0 0" />
     </xacro:aft_fin_macro>
     <xacro:aft_fin_macro namespace="${namespace}" fin_id="3" mesh_filename="${aft_fin_mesh_file}">
-        <!--<origin xyz="-16.583 0.0 2.25677" rpy="${1.0 * pi} 0 0" />-->
-        <origin xyz="-1.537 0 0.136" rpy="${1.0 * pi} 0 0" />
-        <!--<origin xyz="-4.84155 0 0.4284" rpy="${1.0 * pi} 0 0" />-->
+        <!--<origin xyz="-3.4129751 0 0.40526605" rpy="0 0 0" />-->
+        <origin xyz="-3.4129751 0 0.40526605" rpy="${1.0 * pi} 0 0" />
     </xacro:aft_fin_macro>
     <xacro:aft_fin_macro namespace="${namespace}" fin_id="4" mesh_filename="${aft_fin_mesh_file}">
-        <!--<origin xyz="-16.583 -2.2397 -0.4013" rpy="${1.5 * pi} 0 0" />-->
-        <origin xyz="-1.537 -0.136 0" rpy="${1.5 * pi} 0 0" />
-        <!--<origin xyz="-4.84155 -0.4284 0" rpy="${1.5 * pi} 0 0" />-->
+        <!--<origin xyz="-3.4129751 -0.46646423 0.05598445" rpy="${1.0 * pi} 0 0" />-->
+        <!--<origin xyz="-3.4129751 -0.46646423 0.05598445" rpy="${1.5 * pi} 0 0" />-->
+        <origin xyz="-3.4129751 -0.46646423 0.0" rpy="${1.5 * pi} 0 0" />
     </xacro:aft_fin_macro>
     <xacro:aft_fin_macro namespace="${namespace}" fin_id="5" mesh_filename="${aft_fin_mesh_file}">
-        <!--<origin xyz="-16.583 0.0 -2.25677" rpy="${0.0 * pi} 0 0" />-->
-        <origin xyz="-1.537 0 -0.136" rpy="${0.0 * pi} 0 0" />
-        <!--<origin xyz="-4.84155 0 -0.4284" rpy="${0.0 * pi} 0 0" />-->
+        <!--<origin xyz="-3.4129751 0 -0.40526605" rpy="${1.0 * pi} 0 0" />-->
+        <origin xyz="-3.4129751 0 -0.40526605" rpy="${0.0 * pi} 0 0" />
     </xacro:aft_fin_macro>
 </robot>

File: urdf/base.xacro (robot description, xacro)
@@ -28,5 +28,5 @@
               <origin rpy="0 0 0" xyz="0 0 0"/>
               <geometry>
-                  <mesh filename="package://O_29qt/meshes/base_link_ano.STL"/>
+                  <mesh filename="package://O_29qt/meshes/base_link_no_fins.STL"/>
               </geometry>
               <material name="">
@@ -37,5 +37,5 @@
               <origin rpy="0 0 0" xyz="0 0 0"/>
               <geometry>
-                <mesh filename="package://O_29qt/meshes/base_link_ano.STL"/>
+                <mesh filename="package://O_29qt/meshes/base_link_no_fins.STL"/>
               </geometry>
             </collision>
@@ -52,5 +52,5 @@
                   <mesh filename="package://O_29qt/meshes/base_link.STL"/>
                   <mesh filename="package://O_29qt/meshes/QT1.STL"/>
-                  <mesh filename="package://O_29qt/meshes/base_link_ano.STL"/>
+                  <mesh filename="package://O_29qt/meshes/base_link_no_fins.STL"/>
               </geometry>
               <material name="">

File: urdf/gazebo.xacro (robot description, xacro)
@@ -6,5 +6,6 @@
     <!--<xacro:property name="O_29qt_volume" value="${819026 / 9.8 / 1000}"/>-->
     <!--<xacro:property name="O_29qt_volume" value="${838 / 9.8 / 1000}"/>-->
-    <xacro:property name="O_29qt_volume" value="${4690 / 1000}"/>
+    <!--<xacro:property name="O_29qt_volume" value="${4690 / 1000}"/>-->
+    <xacro:property name="O_29qt_volume" value="${4390 / 1000}"/>
     <!-- Describing the dimensions of the vehicle's bounding box -->
     <!--<xacro:property name="O_29qt_length" value="40.97"/>

File: urdf/snippets.xacro (robot description, xacro)
@@ -35,7 +35,7 @@
                 <gain>1</gain>
                 <!-- Maximum allowed input value for the input signal for thruster unit -->
-                <clampMax>2300</clampMax>
+                <clampMax>2500</clampMax>
                 <!-- Minimum allowed input value for the input signal for thruster unit -->
-                <clampMin>-2300</clampMin>
+                <clampMin>-2500</clampMin>
                 <!-- Maximum thrust force output allowed -->
                 <thrustMax>26338.811</thrustMax>
@@ -85,13 +85,16 @@
     <!-- MACRO FOR FIN/RUDDER UNITS  -->
   <!-- A separate mesh for the fin should be stored in the meshes folder -->
-  <xacro:property name="front_fin_mesh_file" value="file://$(find O_29qt)/meshes/front_fin.dae"/>
-  <xacro:property name="aft_fin_mesh_file" value="file://$(find O_29qt)/meshes/aft_fin.dae"/>
+  <!--<xacro:property name="front_fin_mesh_file" value="file://$(find O_29qt)/meshes/front_fin_latest.STL"/>-->
+  <xacro:property name="front_fin_mesh_file" value="file://$(find armsauv_description)/meshes/front_fin.dae"/>
+  <!--<xacro:property name="aft_fin_mesh_file" value="file://$(find O_29qt)/meshes/aft_fin_latest.STL"/>-->
+  <xacro:property name="aft_fin_mesh_file" value="file://$(find armsauv_description)/meshes/aft_fin.dae"/>
   <!-- Fin properties -->
   <xacro:property name="fin_rho" value="1025"/>
   <!--<xacro:property name="front_fin_area" value="2.9153726"/>-->
   <!--<xacro:property name="front_fin_area" value="0.0127"/>-->
-  <xacro:property name="front_fin_area" value="0.785"/>
-  <xacro:property name="front_fin_lift_coefficient" value="20.843"/>
-  <xacro:property name="front_fin_drag_coefficient" value="1.98"/>
+  <xacro:property name="front_fin_area" value="0.116615"/>
+  <!--<xacro:property name="front_fin_lift_coefficient" value="1.668475641"/>-->
+  <xacro:property name="front_fin_lift_coefficient" value="3.416017484"/>
+  <xacro:property name="front_fin_drag_coefficient" value="0.26542681"/>
   <xacro:macro name="front_fin_macro" params="namespace fin_id *origin mesh_filename">
       <xacro:fin_quadratic_macro
@@ -107,10 +110,43 @@
         <xacro:insert_block name="origin"/>
       </xacro:fin_quadratic_macro>
+      <!--<link name="${namespace}/fin${fin_id}">
+          <visual>
+              <origin xyz="0 0 0" rpy="0 0 0"/>
+              <geometry>
+                  <mesh filename="${mesh_filename}" scale="9 9 9"/>
+              </geometry>
+          </visual>
+      </link>
+      <joint name="${namespace}/fin${fin_id}_joint" type="revolute">
+          <limit effort="0" lower="${-30*d2r}" upper="${30*d2r}" velocity="0"/>
+          <xacro:insert_block name="origin"/>
+          <axiz xyz="0 0 1"/>
+          <parent link="${namespace}/base_link"/>
+          <child link="${namespace}/fin${fin_id}"/>
+      </joint>
+      <gazebo>
+          <plugin name="${namespace}_fin${fin_id}_model" filename="libuuv_fin_ros_plugin.so">
+              <dynamics>
+                  <type>FirstOrder</type>
+                  <timeConstant>0.1</timeConstant>
+              </dynamics>
+              <liftdrag>
+                  <type>Quadratic</type>
+                  <lift_constant>${0.5 * fin_rho * front_fin_area * front_fin_lift_coefficient}</lift_constant>
+                  <drag_constant>${0.5 * fin_rho * front_fin_area * front_fin_drag_coefficient}</drag_constant>
+              </liftdrag>
+              <current_velocity_topic>current_velocity</current_velocity_topic>
+              <fin_id>${fin_id}</fin_id>
+              <link_name>${namespace}/fin${fin_id}</link_name>
+              <joint_name>${namespace}/fin${fin_id}_joint</joint_name>
+          </plugin>
+      </gazebo>-->
   </xacro:macro>
   <!--<xacro:property name="aft_fin_area" value="2.656049"/>-->
   <!--<xacro:property name="aft_fin_area" value="0.0172"/>-->
-  <xacro:property name="aft_fin_area" value="0.785"/>
-  <xacro:property name="aft_fin_lift_coefficient" value="19.1395"/>
-  <xacro:property name="aft_fin_drag_coefficient" value="1.98"/>
+  <xacro:property name="aft_fin_area" value="0.106243"/>
+  <!--<xacro:property name="aft_fin_lift_coefficient" value="1.74975211"/>-->
+  <xacro:property name="aft_fin_lift_coefficient" value="3.290443227"/>
+  <xacro:property name="aft_fin_drag_coefficient" value="0.269448395"/>
   <xacro:macro name="aft_fin_macro" params="namespace fin_id *origin mesh_filename">
       <xacro:fin_quadratic_macro
