Commit message: Modify configuration for standard size model

File: urdf/actuators.xacro (robot description, xacro)
@@ -2,33 +2,30 @@
 <robot xmlns:xacro="http://www.ros.org/wiki/xacro">
     <xacro:thruster_macro robot_namespace="${namespace}" thruster_id = "0">
-        <origin xyz="-4.668392 0.0 0" rpy="0 0 0" />
+        <!--<origin xyz="-4.668392 0.0 0" rpy="0 0 0" />-->
+        <origin xyz="-4.56680 0.0 0.0" rpy="0 0 0" />
     </xacro:thruster_macro>
-    <xacro:front_fin_macro namespace="${namespace}" fin_id="0" mesh_filename="${front_fin_mesh_file}">
-        <!--<origin xyz="2.168598 0.4569450 0.27093419" rpy="0 0 0" />-->
-        <!--<origin xyz="2.168598 -0.4569450 0.27093419" rpy="${0.5 * pi} 0 0" />-->
-        <origin xyz="2.168598 -0.4569450 0.0" rpy="${0.5 * pi} 0 0" />
-    </xacro:front_fin_macro>
-    <xacro:front_fin_macro namespace="${namespace}" fin_id="1" mesh_filename="${front_fin_mesh_file}">
-        <!--<origin xyz="2.168598 -0.4569450 0.27093419" rpy="${1.0 * pi} 0 0" />-->
-        <!--<origin xyz="2.168598 0.4569450 0.27093419" rpy="${1.5 * pi} 0 0" />-->
-        <origin xyz="2.168598 0.4569450 0.0" rpy="${1.5 * pi} 0 0" />
-    </xacro:front_fin_macro>
-    <xacro:aft_fin_macro namespace="${namespace}" fin_id="2" mesh_filename="${aft_fin_mesh_file}">
-        <!--<origin xyz="-3.4129751 0.46646423 0.05598445" rpy="0 0 0" />-->
-        <!--<origin xyz="-3.4129751 0.46646423 0.05598445" rpy="${0.5 * pi} 0 0" />-->
-        <origin xyz="-3.4129751 0.46646423 0.0" rpy="${0.5 * pi} 0 0" />
-    </xacro:aft_fin_macro>
-    <xacro:aft_fin_macro namespace="${namespace}" fin_id="3" mesh_filename="${aft_fin_mesh_file}">
+    <xacro:front_left_fin_macro namespace="${namespace}" fin_id="0" mesh_filename="${front_left_fin_mesh_file}">
+        <!--<origin xyz="2.168598 0.4569450 0.0" rpy="0 0 0" />-->
+        <origin xyz="2.18604 0.46068 0.252" rpy="0 0 0" />
+    </xacro:front_left_fin_macro>
+    <xacro:front_right_fin_macro namespace="${namespace}" fin_id="1" mesh_filename="${front_left_fin_mesh_file}">
+        <!--<origin xyz="2.168598 -0.4569450 0.0" rpy="0 0 0" />-->
+        <origin xyz="2.18604 -0.46068 0.252" rpy="0 0 0" />
+    </xacro:front_right_fin_macro>
+    <xacro:front_left_fin_macro namespace="${namespace}" fin_id="2" mesh_filename="${front_left_fin_mesh_file}">
+        <!--<origin xyz="-3.4129751 0.46646423 0.0" rpy="0 0 0" />-->
+        <origin xyz="-3.44858 0.41165 0.08295" rpy="0 0 0" />
+    </xacro:front_left_fin_macro>
+    <xacro:back_up_fin_macro namespace="${namespace}" fin_id="3" mesh_filename="${back_up_fin_mesh_file}">
         <!--<origin xyz="-3.4129751 0 0.40526605" rpy="0 0 0" />-->
-        <origin xyz="-3.4129751 0 0.40526605" rpy="${1.0 * pi} 0 0" />
-    </xacro:aft_fin_macro>
-    <xacro:aft_fin_macro namespace="${namespace}" fin_id="4" mesh_filename="${aft_fin_mesh_file}">
-        <!--<origin xyz="-3.4129751 -0.46646423 0.05598445" rpy="${1.0 * pi} 0 0" />-->
-        <!--<origin xyz="-3.4129751 -0.46646423 0.05598445" rpy="${1.5 * pi} 0 0" />-->
-        <origin xyz="-3.4129751 -0.46646423 0.0" rpy="${1.5 * pi} 0 0" />
-    </xacro:aft_fin_macro>
-    <xacro:aft_fin_macro namespace="${namespace}" fin_id="5" mesh_filename="${aft_fin_mesh_file}">
-        <!--<origin xyz="-3.4129751 0 -0.40526605" rpy="${1.0 * pi} 0 0" />-->
-        <origin xyz="-3.4129751 0 -0.40526605" rpy="${0.0 * pi} 0 0" />
-    </xacro:aft_fin_macro>
+        <origin xyz="-3.44814 0 0.40858" rpy="0 0 0" />
+    </xacro:back_up_fin_macro>
+    <xacro:front_right_fin_macro namespace="${namespace}" fin_id="4" mesh_filename="${front_left_fin_mesh_file}">
+        <!--<origin xyz="-3.4129751 -0.46646423 0.0" rpy="0 0 0" />-->
+        <origin xyz="-3.44858 -0.41165 0.08295" rpy="0 0 0" />
+    </xacro:front_right_fin_macro>
+    <xacro:back_down_fin_macro namespace="${namespace}" fin_id="5" mesh_filename="${back_down_fin_mesh_file}">
+        <!--<origin xyz="-3.4129751 0 -0.40526605" rpy="0 0 0" />-->
+        <origin xyz="-3.44814 0 -0.40858" rpy="0 0 0" />
+    </xacro:back_down_fin_macro>
 </robot>

File: urdf/base.xacro (robot description, xacro)
@@ -28,5 +28,6 @@
               <origin rpy="0 0 0" xyz="0 0 0"/>
               <geometry>
-                  <mesh filename="package://O_29qt/meshes/O_29_base.dae"/>
+                  <!--<mesh filename="package://O_29qt/meshes/0.21/O_29_base_0.21.dae" scale="1 1 1"/>-->
+                  <mesh filename="package://O_29qt/meshes/O_29_base.dae" scale="0.21 0.21 0.21"/>
               </geometry>
               <material name="">
@@ -37,5 +38,6 @@
               <origin rpy="0 0 0" xyz="0 0 0"/>
               <geometry>
-                <mesh filename="package://O_29qt/meshes/O_29_base.dae"/>
+                  <!--<mesh filename="package://O_29qt/meshes/0.21/O_29_base_0.21.dae" scale="1 1 1"/>-->
+                  <mesh filename="package://O_29qt/meshes/O_29_base.dae" scale="0.21 0.21 0.21"/>
               </geometry>
             </collision>

File: urdf/gazebo.xacro (robot description, xacro)
@@ -115,10 +115,10 @@
           <type>fossen</type>
           <added_mass>
-              ${-xudot*D3*0.1}      ${-xvdot*D3*0.1}       ${-xwdot*D3*0.1}       ${-xpdot*D4*0.1}      ${-xqdot*D4*0.1}      ${-xrdot*D4*0.1}
-              ${-yudot*D3*0.1}      ${-yvdot*D3*0.1}       ${-ywdot*D3*0.1}       ${-ypdot*D4*0.1}      ${-yqdot*D4*0.1}      ${-yrdot*D4*0.1}
-              ${-zudot*D3*0.1}      ${-zvdot*D3*0.1}       ${-zwdot*D3*0.1}       ${-zpdot*D4*0.1}      ${-zqdot*D4*0.1}      ${-zrdot*D4*0.1}
-              ${-kudot*D4*0.1}      ${-kvdot*D4*0.1}       ${-kwdot*D4*0.1}       ${-kpdot*D5*0.1}      ${-kqdot*D5*0.1}      ${-krdot*D5*0.1}
-              ${-mudot*D4*0.1}      ${-mvdot*D4*0.1}       ${-mwdot*D4*0.1}       ${-mpdot*D5*0.1}      ${-mqdot*D5*0.1}      ${-mrdot*D5*0.1}
-              ${-nudot*D4*0.1}      ${-nvdot*D4*0.1}       ${-nwdot*D4*0.1}       ${-npdot*D5*0.1}      ${-nqdot*D5*0.1}      ${-nrdot*D5*0.1}
+              ${xudot*D3*0.1}      ${xvdot*D3*0.1}       ${xwdot*D3*0.1}       ${xpdot*D4*0.1}      ${xqdot*D4*0.1}      ${-xrdot*D4*0.1}
+              ${yudot*D3*0.1}      ${yvdot*D3*0.1}       ${ywdot*D3*0.1}       ${ypdot*D4*0.1}      ${yqdot*D4*0.1}      ${-yrdot*D4*0.1}
+              ${zudot*D3*0.1}      ${zvdot*D3*0.1}       ${zwdot*D3*0.1}       ${zpdot*D4*0.1}      ${zqdot*D4*0.1}      ${-zrdot*D4*0.1}
+              ${kudot*D4*0.1}      ${kvdot*D4*0.1}       ${kwdot*D4*0.1}       ${kpdot*D5*0.1}      ${kqdot*D5*0.1}      ${-krdot*D5*0.1}
+              ${mudot*D4*0.1}      ${mvdot*D4*0.1}       ${mwdot*D4*0.1}       ${mpdot*D5*0.1}      ${mqdot*D5*0.1}      ${-mrdot*D5*0.1}
+              ${nudot*D4*0.1}      ${nvdot*D4*0.1}       ${nwdot*D4*0.1}       ${npdot*D5*0.1}      ${nqdot*D5*0.1}      ${-nrdot*D5*0.1}
           </added_mass>
           <!--<added_mass>
@@ -155,5 +155,4 @@
             ${muu*D3}      ${muv*D3}       ${muw*D3}       ${mup*D4}      ${muq*D4}      ${mur*D4}
             ${nuu*D3}      ${nuv*D3}       ${nuw*D3}       ${nup*D4}      ${nuq*D4}      ${nur*D4}
-          </quadratic_damping>
           </linear_damping_forward_speed>
           <!--

File: urdf/snippets.xacro (robot description, xacro)
@@ -1,10 +1,10 @@
 <?xml version="1.0" encoding="UTF-8"?>
 <robot xmlns:xacro="http://www.ros.org/wiki/xacro">
-    <xacro:property name="propeller_mesh_file" value="file://$(find O_29qt)/meshes/propeller.STL" />
+    <xacro:property name="propeller_mesh_file" value="file://$(find O_29qt)/meshes/propeller.dae" />
     <xacro:macro name="thruster_macro" params="robot_namespace thruster_id *origin">
         <link name="${robot_namespace}/thruster_${thruster_id}">
             <visual>
                 <geometry>
-                    <mesh filename="${propeller_mesh_file}" scale="1 1 1" />
+                    <mesh filename="${propeller_mesh_file}" scale="0.2 0.2 0.2" />
                 </geometry>
             </visual>
@@ -85,18 +85,18 @@
     <!-- MACRO FOR FIN/RUDDER UNITS  -->
   <!-- A separate mesh for the fin should be stored in the meshes folder -->
-  <xacro:property name="front_fin_mesh_file" value="file://$(find O_29qt)/meshes/front_fin_latest.STL"/>
-  <!--<xacro:property name="front_fin_mesh_file" value="file://$(find armsauv_description)/meshes/front_fin.dae"/>-->
-  <xacro:property name="aft_fin_mesh_file" value="file://$(find O_29qt)/meshes/aft_fin_latest.STL"/>
-  <!--<xacro:property name="aft_fin_mesh_file" value="file://$(find armsauv_description)/meshes/aft_fin.dae"/>-->
+  <xacro:property name="front_left_fin_mesh_file" value="file://$(find O_29qt)/meshes/0.21/front_fin_left_0.21.dae"/>
+  <xacro:property name="front_right_fin_mesh_file" value="file://$(find O_29qt)/meshes/0.21/front_fin_right_rev_0.21.dae"/>
+  <xacro:property name="back_up_fin_mesh_file" value="file://$(find O_29qt)/meshes/0.21/back_fin_up_0.21.dae"/>
+  <xacro:property name="back_down_fin_mesh_file" value="file://$(find O_29qt)/meshes/0.21/back_fin_down_0.21.dae"/>
   <!-- Fin properties -->
   <xacro:property name="fin_rho" value="1025"/>
-  <!--<xacro:property name="front_fin_area" value="2.9153726"/>-->
   <!--<xacro:property name="front_fin_area" value="0.0127"/>-->
   <xacro:property name="front_fin_area" value="0.116615"/>
-  <!--<xacro:property name="front_fin_lift_coefficient" value="1.668475641"/>-->
   <xacro:property name="front_fin_lift_coefficient" value="3.416017484"/>
   <xacro:property name="front_fin_drag_coefficient" value="0.26542681"/>
-  <xacro:macro name="front_fin_macro" params="namespace fin_id *origin mesh_filename">
-      <!--<xacro:fin_quadratic_macro
+  <!--<xacro:property name="front_fin_lift_coefficient" value="20.843"/>-->
+  <!--<xacro:property name="front_fin_drag_coefficient" value="1.98"/>-->
+  <xacro:macro name="front_left_fin_macro" params="namespace fin_id *origin mesh_filename">
+      <xacro:hor_left_fin_quadratic_macro
         namespace="${namespace}"
         parent_link="${namespace}/base_link" fin_id="${fin_id}"
@@ -109,47 +109,29 @@
         current_velocity_topic="current_velocity">
         <xacro:insert_block name="origin"/>
-      </xacro:fin_quadratic_macro>-->
-      <link name="${namespace}/fin${fin_id}">
-          <xacro:no_inertial/>
-          <visual>
-              <origin xyz="0 0 0" rpy="0 0 0"/>
-              <geometry>
-                  <mesh filename="${mesh_filename}" scale="1 1 1"/>
-              </geometry>
-          </visual>
-      </link>
-      <joint name="${namespace}/fin${fin_id}_joint" type="revolute">
-          <limit effort="0" lower="${-90*d2r}" upper="${90*d2r}" velocity="0"/>
-          <xacro:insert_block name="origin"/>
-          <axiz xyz="0 0 1"/>
-          <parent link="${namespace}/base_link"/>
-          <child link="${namespace}/fin${fin_id}"/>
-      </joint>
-      <gazebo>
-          <plugin name="${namespace}_fin${fin_id}_model" filename="libuuv_fin_ros_plugin.so">
-              <dynamics>
-                  <type>FirstOrder</type>
-                  <timeConstant>0.2</timeConstant>
-              </dynamics>
-              <liftdrag>
-                  <type>Quadratic</type>
-                  <lift_constant>${0.5 * fin_rho * front_fin_area * front_fin_lift_coefficient}</lift_constant>
-                  <drag_constant>${0.5 * fin_rho * front_fin_area * front_fin_drag_coefficient}</drag_constant>
-              </liftdrag>
-              <current_velocity_topic>current_velocity</current_velocity_topic>
-              <fin_id>${fin_id}</fin_id>
-              <link_name>${namespace}/fin${fin_id}</link_name>
-              <joint_name>${namespace}/fin${fin_id}_joint</joint_name>
-          </plugin>
-      </gazebo>
+      </xacro:hor_left_fin_quadratic_macro>
+  </xacro:macro>
+  <xacro:macro name="front_right_fin_macro" params="namespace fin_id *origin mesh_filename">
+      <xacro:hor_right_fin_quadratic_macro
+        namespace="${namespace}"
+        parent_link="${namespace}/base_link" fin_id="${fin_id}"
+        min_joint_limit="${-90.0 * d2r}"
+        max_joint_limit="${90.0 * d2r}"
+        mesh_filename="${mesh_filename}"
+        fin_dynamics_time_constant="0.2"
+        lift_constant="${0.5 * fin_rho * front_fin_area * front_fin_lift_coefficient}"
+        drag_constant="${0.5 * fin_rho * front_fin_area * front_fin_drag_coefficient}"
+        current_velocity_topic="current_velocity">
+        <xacro:insert_block name="origin"/>
+      </xacro:hor_right_fin_quadratic_macro>
   </xacro:macro>
   <!--<xacro:property name="aft_fin_area" value="2.656049"/>-->
   <!--<xacro:property name="aft_fin_area" value="0.0172"/>-->
   <xacro:property name="aft_fin_area" value="0.106243"/>
-  <!--<xacro:property name="aft_fin_lift_coefficient" value="1.74975211"/>-->
   <xacro:property name="aft_fin_lift_coefficient" value="3.290443227"/>
   <xacro:property name="aft_fin_drag_coefficient" value="0.269448395"/>
-  <xacro:macro name="aft_fin_macro" params="namespace fin_id *origin mesh_filename">
-      <!--<xacro:fin_quadratic_macro
+  <!--<xacro:property name="aft_fin_lift_coefficient" value="19.1395"/>-->
+  <!--<xacro:property name="aft_fin_drag_coefficient" value="1.98"/>-->
+  <xacro:macro name="back_up_fin_macro" params="namespace fin_id *origin mesh_filename">
+      <xacro:lat_up_fin_quadratic_macro
         namespace="${namespace}"
         parent_link="${namespace}/base_link"
@@ -163,38 +145,20 @@
         current_velocity_topic="current_velocity">
         <xacro:insert_block name="origin"/>
-      </xacro:fin_quadratic_macro>-->
-      <link name="${namespace}/fin${fin_id}">
-          <xacro:no_inertial/>
-          <visual>
-              <origin xyz="0 0 0" rpy="0 0 0"/>
-              <geometry>
-                  <mesh filename="${mesh_filename}" scale="1 1 1"/>
-              </geometry>
-          </visual>
-      </link>
-      <joint name="${namespace}/fin${fin_id}_joint" type="revolute">
-          <limit effort="0" lower="${-90*d2r}" upper="${90*d2r}" velocity="0"/>
-          <xacro:insert_block name="origin"/>
-          <axiz xyz="0 0 1"/>
-          <parent link="${namespace}/base_link"/>
-          <child link="${namespace}/fin${fin_id}"/>
-      </joint>
-      <gazebo>
-          <plugin name="${namespace}_fin${fin_id}_model" filename="libuuv_fin_ros_plugin.so">
-              <dynamics>
-                  <type>FirstOrder</type>
-                  <timeConstant>0.2</timeConstant>
-              </dynamics>
-              <liftdrag>
-                  <type>Quadratic</type>
-                  <lift_constant>${0.5 * fin_rho * front_fin_area * front_fin_lift_coefficient}</lift_constant>
-                  <drag_constant>${0.5 * fin_rho * front_fin_area * front_fin_drag_coefficient}</drag_constant>
-              </liftdrag>
-              <current_velocity_topic>current_velocity</current_velocity_topic>
-              <fin_id>${fin_id}</fin_id>
-              <link_name>${namespace}/fin${fin_id}</link_name>
-              <joint_name>${namespace}/fin${fin_id}_joint</joint_name>
-          </plugin>
-      </gazebo>
+      </xacro:lat_up_fin_quadratic_macro>
+  </xacro:macro>
+  <xacro:macro name="back_down_fin_macro" params="namespace fin_id *origin mesh_filename">
+      <xacro:lat_down_fin_quadratic_macro
+        namespace="${namespace}"
+        parent_link="${namespace}/base_link"
+        fin_id="${fin_id}"
+        min_joint_limit="${-90.0 * d2r}"
+        max_joint_limit="${90.0 * d2r}"
+        mesh_filename="${mesh_filename}"
+        fin_dynamics_time_constant="0.2"
+        lift_constant="${0.5 * fin_rho * aft_fin_area * aft_fin_lift_coefficient}"
+        drag_constant="${0.5 * fin_rho * aft_fin_area * aft_fin_drag_coefficient}"
+        current_velocity_topic="current_velocity">
+        <xacro:insert_block name="origin"/>
+      </xacro:lat_down_fin_quadratic_macro>
   </xacro:macro>
   <!-- <xacro:macro name="fin_macro" params="namespace fin_id *origin mesh_filename">
