Commit message: Test hydrodynamic params of standard model

File: urdf/actuators.xacro (robot description, xacro)
@@ -2,30 +2,42 @@
 <robot xmlns:xacro="http://www.ros.org/wiki/xacro">
     <xacro:thruster_macro robot_namespace="${namespace}" thruster_id = "0">
-        <!--<origin xyz="-4.668392 0.0 0" rpy="0 0 0" />-->
         <origin xyz="-4.56680 0.0 0.0" rpy="0 0 0" />
     </xacro:thruster_macro>
-    <xacro:front_left_fin_macro namespace="${namespace}" fin_id="0" mesh_filename="${front_left_fin_mesh_file}">
-        <!--<origin xyz="2.168598 0.4569450 0.0" rpy="0 0 0" />-->
+    <!--<xacro:front_left_fin_macro namespace="${namespace}" fin_id="0" mesh_filename="${front_left_fin_mesh_file}">
         <origin xyz="2.18604 0.46068 0.252" rpy="0 0 0" />
     </xacro:front_left_fin_macro>
     <xacro:front_right_fin_macro namespace="${namespace}" fin_id="1" mesh_filename="${front_left_fin_mesh_file}">
-        <!--<origin xyz="2.168598 -0.4569450 0.0" rpy="0 0 0" />-->
         <origin xyz="2.18604 -0.46068 0.252" rpy="0 0 0" />
     </xacro:front_right_fin_macro>
-    <xacro:front_left_fin_macro namespace="${namespace}" fin_id="2" mesh_filename="${front_left_fin_mesh_file}">
-        <!--<origin xyz="-3.4129751 0.46646423 0.0" rpy="0 0 0" />-->
+    <xacro:back_left_fin_macro namespace="${namespace}" fin_id="2" mesh_filename="${back_left_fin_mesh_file}">
         <origin xyz="-3.44858 0.41165 0.08295" rpy="0 0 0" />
-    </xacro:front_left_fin_macro>
+    </xacro:back_left_fin_macro>
     <xacro:back_up_fin_macro namespace="${namespace}" fin_id="3" mesh_filename="${back_up_fin_mesh_file}">
-        <!--<origin xyz="-3.4129751 0 0.40526605" rpy="0 0 0" />-->
         <origin xyz="-3.44814 0 0.40858" rpy="0 0 0" />
     </xacro:back_up_fin_macro>
-    <xacro:front_right_fin_macro namespace="${namespace}" fin_id="4" mesh_filename="${front_left_fin_mesh_file}">
-        <!--<origin xyz="-3.4129751 -0.46646423 0.0" rpy="0 0 0" />-->
+    <xacro:back_right_fin_macro namespace="${namespace}" fin_id="4" mesh_filename="${back_left_fin_mesh_file}">
         <origin xyz="-3.44858 -0.41165 0.08295" rpy="0 0 0" />
-    </xacro:front_right_fin_macro>
+    </xacro:back_right_fin_macro>
     <xacro:back_down_fin_macro namespace="${namespace}" fin_id="5" mesh_filename="${back_down_fin_mesh_file}">
-        <!--<origin xyz="-3.4129751 0 -0.40526605" rpy="0 0 0" />-->
         <origin xyz="-3.44814 0 -0.40858" rpy="0 0 0" />
-    </xacro:back_down_fin_macro>
+    </xacro:back_down_fin_macro>-->
+    <!-- Instantiate fins, if necessary -->
+    <xacro:front_fin_macro namespace="${namespace}" fin_id="0" mesh_filename="${backup_front_fin_mesh_file}">
+        <origin xyz="2.18604 -0.46068 0.252" rpy="${0.5 * pi} 0 0" />
+    </xacro:front_fin_macro>
+    <xacro:front_fin_macro namespace="${namespace}" fin_id="1" mesh_filename="${backup_front_fin_mesh_file}">
+        <origin xyz="2.18604 0.46068 0.252" rpy="${1.5 * pi} 0 0" />
+    </xacro:front_fin_macro>
+    <xacro:aft_fin_macro namespace="${namespace}" fin_id="2" mesh_filename="${backup_back_fin_mesh_file}">
+        <origin xyz="-3.44858 0.41165 0.08295" rpy="${0.5 * pi}  0 0" />
+    </xacro:aft_fin_macro>
+    <xacro:aft_fin_macro namespace="${namespace}" fin_id="3" mesh_filename="${backup_back_fin_mesh_file}">
+        <origin xyz="-3.44814 0 0.40858" rpy="${1 * pi} 0 0" />
+    </xacro:aft_fin_macro>
+    <xacro:aft_fin_macro namespace="${namespace}" fin_id="4" mesh_filename="${backup_back_fin_mesh_file}">
+        <origin xyz="-3.44858 -0.41165 0.08295" rpy="${1.5 * pi} 0 0" />
+    </xacro:aft_fin_macro>
+    <xacro:aft_fin_macro namespace="${namespace}" fin_id="5" mesh_filename="${backup_back_fin_mesh_file}">
+        <origin xyz="-3.44814 0 -0.40858" rpy="${0 * pi} 0 0" />
+    </xacro:aft_fin_macro>
 </robot>

File: urdf/gazebo.xacro (robot description, xacro)
@@ -8,7 +8,7 @@
     <!-- Added base parameters -->
     <xacro:property name="O_29qt_length" value="8.534"/>
-    <xacro:property name="O_29qt_width"  value="1.0256"/>
+    <xacro:property name="O_29qt_width"  value="1.6568"/>
     <xacro:property name="O_29qt_radius"  value="0.5128"/>
-    <xacro:property name="O_29qt_height" value="1.0256"/>
+    <xacro:property name="O_29qt_height" value="1.5749"/>
     <xacro:property name="rho" value="1025" />
     <xacro:property name="D0" value="${rho * 0.5}"/>
@@ -123,10 +123,10 @@
           </added_mass>
           <!--<added_mass>
-            1.432   0       0       0     0      0
-            0    120.645    0       0     0    4.895
-            0       0    130.513    0  -16.488   0
-            0       0       0    0.386    0      0
-            0       0   -16.488     0  78.266    0
-            0     4.895     0       0     0    67.489
+              ${xudot*D3*0.1}            0.0                   0.0                  0.0                  0.0                    0.0
+                    0.0            ${yvdot*D3*0.1}             0.0                  0.0                  0.0             ${-yrdot*D4*0.1}
+                    0.0                  0.0             ${zwdot*D3*0.1}            0.0             ${zqdot*D4*0.1}             0.0
+                    0.0                  0.0                   0.0             ${kpdot*D5*0.1}           0.0                    0.0
+                    0.0                  0.0             ${mwdot*D4*0.1}            0.0             ${mqdot*D5*0.1}             0.0
+                    0.0            ${nvdot*D4*0.1}             0.0                  0.0                  0.0             ${-nrdot*D5*0.1}
           </added_mass>-->
           <!--
@@ -156,4 +156,12 @@
             ${nuu*D3}      ${nuv*D3}       ${nuw*D3}       ${nup*D4}      ${nuq*D4}      ${nur*D4}
           </linear_damping_forward_speed>
+          <!--<linear_damping_forward_speed>
+            ${xuu*D2}         0.0             0.0             0.0             0.0            0.0
+                0.0        ${yuv*D2}          0.0             0.0             0.0        ${yur*D3}
+                0.0           0.0          ${zuw*D2}          0.0         ${zuq*D3}          0.0
+                0.0           0.0             0.0          ${kup*D4}          0.0            0.0
+                0.0           0.0          ${muw*D3}          0.0         ${muq*D4}          0.0
+                0.0        ${nuv*D3}          0.0             0.0             0.0        ${nur*D4}
+          </linear_damping_forward_speed>-->
           <!--
             The quadratic damping coefficients can be provided as a diagonal (6 elements)
@@ -161,10 +169,10 @@
           -->
           <!--<quadratic_damping>
-            -3.9     0      0      0     0      0
-              0  -373.287   0      0     0   -4.204
-              0      0  -489.07    0  23.016    0
-              0      0      0   -0.117   0      0
-              0      0   23.342    0 -353.406   0
-              0   0.419     0      0     0  -227.024
+            ${xuu*D2}      ${xuv*D2}       ${xuw*D2}       ${xup*D3}      ${xuq*D3}      ${xur*D3}
+            ${yuu*D2}      ${yuv*D2}       ${yuw*D2}       ${yup*D3}      ${yuq*D3}      ${yur*D3}
+            ${zuu*D2}      ${zuv*D2}       ${zuw*D2}       ${zup*D3}      ${zuq*D3}      ${zur*D3}
+            ${kuu*D3}      ${kuv*D3}       ${kuw*D3}       ${kup*D4}      ${kuq*D4}      ${kur*D4}
+            ${muu*D3}      ${muv*D3}       ${muw*D3}       ${mup*D4}      ${muq*D4}      ${mur*D4}
+            ${nuu*D3}      ${nuv*D3}       ${nuw*D3}       ${nup*D4}      ${nuq*D4}      ${nur*D4}
           </quadratic_damping>-->
         </hydrodynamic_model>

File: urdf/snippets.xacro (robot description, xacro)
@@ -87,14 +87,19 @@
   <xacro:property name="front_left_fin_mesh_file" value="file://$(find O_29qt)/meshes/0.21/front_fin_left_0.21.dae"/>
   <xacro:property name="front_right_fin_mesh_file" value="file://$(find O_29qt)/meshes/0.21/front_fin_right_rev_0.21.dae"/>
+  <xacro:property name="back_left_fin_mesh_file" value="file://$(find O_29qt)/meshes/0.21/back_fin_left_0.21.dae"/>
+  <xacro:property name="back_right_fin_mesh_file" value="file://$(find O_29qt)/meshes/0.21/back_fin_right_0.21.dae"/>
   <xacro:property name="back_up_fin_mesh_file" value="file://$(find O_29qt)/meshes/0.21/back_fin_up_0.21.dae"/>
   <xacro:property name="back_down_fin_mesh_file" value="file://$(find O_29qt)/meshes/0.21/back_fin_down_0.21.dae"/>
+  <xacro:property name="backup_front_fin_mesh_file" value="file://$(find armsauv_description)/meshes/front_fin.dae"/>
+  <xacro:property name="backup_back_fin_mesh_file" value="file://$(find armsauv_description)/meshes/aft_fin.dae"/>
   <!-- Fin properties -->
   <xacro:property name="fin_rho" value="1025"/>
   <!--<xacro:property name="front_fin_area" value="0.0127"/>-->
   <xacro:property name="front_fin_area" value="0.116615"/>
-  <xacro:property name="front_fin_lift_coefficient" value="3.416017484"/>
+  <!--<xacro:property name="front_fin_lift_coefficient" value="3.416017484"/>-->
+  <!--<xacro:property name="front_fin_lift_coefficient" value="1.668475641"/>
+  <xacro:property name="front_fin_drag_coefficient" value="0.26542681"/>-->
+  <xacro:property name="front_fin_lift_coefficient" value="1.668475641"/>
   <xacro:property name="front_fin_drag_coefficient" value="0.26542681"/>
-  <!--<xacro:property name="front_fin_lift_coefficient" value="20.843"/>-->
-  <!--<xacro:property name="front_fin_drag_coefficient" value="1.98"/>-->
   <xacro:macro name="front_left_fin_macro" params="namespace fin_id *origin mesh_filename">
       <xacro:hor_left_fin_quadratic_macro
@@ -128,8 +133,37 @@
   <!--<xacro:property name="aft_fin_area" value="0.0172"/>-->
   <xacro:property name="aft_fin_area" value="0.106243"/>
-  <xacro:property name="aft_fin_lift_coefficient" value="3.290443227"/>
+  <!--<xacro:property name="aft_fin_lift_coefficient" value="3.290443227"/>
+  <xacro:property name="aft_fin_drag_coefficient" value="0.269448395"/>-->
+  <xacro:property name="aft_fin_lift_coefficient" value="1.74975211"/>
   <xacro:property name="aft_fin_drag_coefficient" value="0.269448395"/>
-  <!--<xacro:property name="aft_fin_lift_coefficient" value="19.1395"/>-->
-  <!--<xacro:property name="aft_fin_drag_coefficient" value="1.98"/>-->
+  <xacro:macro name="back_left_fin_macro" params="namespace fin_id *origin mesh_filename"> <xacro:hor_left_fin_quadratic_macro
+        namespace="${namespace}"
+        parent_link="${namespace}/base_link"
+        fin_id="${fin_id}"
+        min_joint_limit="${-90.0 * d2r}"
+        max_joint_limit="${90.0 * d2r}"
+        mesh_filename="${mesh_filename}"
+        fin_dynamics_time_constant="0.2"
+        lift_constant="${0.5 * fin_rho * aft_fin_area * aft_fin_lift_coefficient}"
+        drag_constant="${0.5 * fin_rho * aft_fin_area * aft_fin_drag_coefficient}"
+        current_velocity_topic="current_velocity">
+        <xacro:insert_block name="origin"/>
+      </xacro:hor_left_fin_quadratic_macro>
+  </xacro:macro>
+  <xacro:macro name="back_right_fin_macro" params="namespace fin_id *origin mesh_filename">
+      <xacro:hor_right_fin_quadratic_macro
+        namespace="${namespace}"
+        parent_link="${namespace}/base_link"
+        fin_id="${fin_id}"
+        min_joint_limit="${-90.0 * d2r}"
+        max_joint_limit="${90.0 * d2r}"
+        mesh_filename="${mesh_filename}"
+        fin_dynamics_time_constant="0.2"
+        lift_constant="${0.5 * fin_rho * aft_fin_area * aft_fin_lift_coefficient}"
+        drag_constant="${0.5 * fin_rho * aft_fin_area * aft_fin_drag_coefficient}"
+        current_velocity_topic="current_velocity">
+        <xacro:insert_block name="origin"/>
+      </xacro:hor_right_fin_quadratic_macro>
+  </xacro:macro>
   <xacro:macro name="back_up_fin_macro" params="namespace fin_id *origin mesh_filename">
       <xacro:lat_up_fin_quadratic_macro
@@ -162,47 +196,33 @@
       </xacro:lat_down_fin_quadratic_macro>
   </xacro:macro>
-  <!-- <xacro:macro name="fin_macro" params="namespace fin_id *origin mesh_filename">
-      <xacro:fin_two_lines_macro
-        namespace="${namespace}"
-        parent_link="${namespace}/base_link"
-        fin_id="${fin_id}"
-        min_joint_limit="${-80*d2r}"
-        max_joint_limit="${80*d2r}"
-        mesh_filename="${mesh_filename}"
-        fin_dynamics_time_constant="0.1"
-        fin_cross_section_area="${fin_area}"
-        current_velocity_topic="current_velocity"
-        fluid_density="1025.0"
-        a0="0.0"
-        alpha_stall="1.57"
-        cla="${0.5 * fin_rho * fin_area * fin_lift_coefficient}"
-        cla_stall="0.0"
-        cda="${0.5 * fin_rho * fin_area * fin_drag_coefficient}"
-        cda_stall="0">
-        <xacro:insert_block name="origin"/>
-      </xacro:fin_two_lines_macro>
-    </xacro:macro> -->
-    <!-- <xacro:macro name="fin_macro" params="namespace fin_id *origin mesh_filename">
-      <xacro:fin_two_lines_macro
-        namespace="${namespace}"
-        parent_link="${namespace}/base_link"
-        fin_id="${fin_id}"
-        min_joint_limit="${-80*d2r}"
-        max_joint_limit="${80*d2r}"
-        mesh_filename="${mesh_filename}"
-        fin_dynamics_time_constant="0.1"
-        fin_cross_section_area="${fin_area}"
-        current_velocity_topic="current_velocity"
-        fluid_density="1025.0"
-        a0="0.0"
-        alpha_stall="0.436332313"
-        cla="2.435070629"
-        cla_stall="0"
-        cda="0"
-        cda_stall="0">
-        <xacro:insert_block name="origin"/>
-      </xacro:fin_two_lines_macro>
-    </xacro:macro> -->
-    <!-- cla_stall="-1.929963096"
-        cda="1.101841914" -->
+  <xacro:macro name="front_fin_macro" params="namespace fin_id *origin mesh_filename">
+      <xacro:fin_quadratic_macro
+        namespace="${namespace}"
+        parent_link="${namespace}/base_link"
+        fin_id="${fin_id}"
+        min_joint_limit="${-90.0 * d2r}"
+        max_joint_limit="${90.0 * d2r}"
+        mesh_filename="${mesh_filename}"
+        fin_dynamics_time_constant="0.2"
+        lift_constant="${0.5 * fin_rho * front_fin_area * front_fin_lift_coefficient}"
+        drag_constant="${0.5 * fin_rho * front_fin_area * front_fin_drag_coefficient}"
+        current_velocity_topic="current_velocity">
+        <xacro:insert_block name="origin"/>
+      </xacro:fin_quadratic_macro>
+  </xacro:macro>
+  <xacro:macro name="aft_fin_macro" params="namespace fin_id *origin mesh_filename">
+      <xacro:fin_quadratic_macro
+        namespace="${namespace}"
+        parent_link="${namespace}/base_link"
+        fin_id="${fin_id}"
+        min_joint_limit="${-90.0 * d2r}"
+        max_joint_limit="${90.0 * d2r}"
+        mesh_filename="${mesh_filename}"
+        fin_dynamics_time_constant="0.2"
+        lift_constant="${0.5 * fin_rho * aft_fin_area * aft_fin_lift_coefficient}"
+        drag_constant="${0.5 * fin_rho * aft_fin_area * aft_fin_drag_coefficient}"
+        current_velocity_topic="current_velocity">
+        <xacro:insert_block name="origin"/>
+      </xacro:fin_quadratic_macro>
+  </xacro:macro>
 </robot>

Commit message: Reset mesh file paths and position of actuators

File: urdf/actuators.xacro (robot description, xacro)
@@ -23,21 +23,21 @@
     </xacro:back_down_fin_macro>-->
     <!-- Instantiate fins, if necessary -->
-    <xacro:front_fin_macro namespace="${namespace}" fin_id="0" mesh_filename="${backup_front_fin_mesh_file}">
-        <origin xyz="2.18604 -0.46068 0.252" rpy="${0.5 * pi} 0 0" />
+    <xacro:front_fin_macro namespace="${namespace}" fin_id="0" mesh_filename="${front_right_fin_mesh_file}">
+        <origin xyz="2.18604 -0.46068 0.252" rpy="${-0.5 * pi} 0 0" />
     </xacro:front_fin_macro>
-    <xacro:front_fin_macro namespace="${namespace}" fin_id="1" mesh_filename="${backup_front_fin_mesh_file}">
-        <origin xyz="2.18604 0.46068 0.252" rpy="${1.5 * pi} 0 0" />
+    <xacro:front_fin_macro namespace="${namespace}" fin_id="1" mesh_filename="${front_left_fin_mesh_file}">
+        <origin xyz="2.18604 0.46068 0.252" rpy="${-0.5 * pi} 0 0" />
     </xacro:front_fin_macro>
-    <xacro:aft_fin_macro namespace="${namespace}" fin_id="2" mesh_filename="${backup_back_fin_mesh_file}">
-        <origin xyz="-3.44858 0.41165 0.08295" rpy="${0.5 * pi}  0 0" />
-    </xacro:aft_fin_macro>
-    <xacro:aft_fin_macro namespace="${namespace}" fin_id="3" mesh_filename="${backup_back_fin_mesh_file}">
-        <origin xyz="-3.44814 0 0.40858" rpy="${1 * pi} 0 0" />
-    </xacro:aft_fin_macro>
-    <xacro:aft_fin_macro namespace="${namespace}" fin_id="4" mesh_filename="${backup_back_fin_mesh_file}">
-        <origin xyz="-3.44858 -0.41165 0.08295" rpy="${1.5 * pi} 0 0" />
-    </xacro:aft_fin_macro>
-    <xacro:aft_fin_macro namespace="${namespace}" fin_id="5" mesh_filename="${backup_back_fin_mesh_file}">
+    <xacro:back_fin_macro namespace="${namespace}" fin_id="2" mesh_filename="${back_up_fin_mesh_file}">
+        <origin xyz="-3.44858 -0.41165 0.08295" rpy="${0.5 * pi}  0 0" />
+    </xacro:back_fin_macro>
+    <xacro:back_fin_macro namespace="${namespace}" fin_id="3" mesh_filename="${back_up_fin_mesh_file}">
+        <origin xyz="-3.44814 0 0.40858" rpy="${0 * pi} 0 0" />
+    </xacro:back_fin_macro>
+    <xacro:back_fin_macro namespace="${namespace}" fin_id="4" mesh_filename="${back_down_fin_mesh_file}">
+        <origin xyz="-3.44858 0.41165 0.08295" rpy="${0.5 * pi} 0 0" />
+    </xacro:back_fin_macro>
+    <xacro:back_fin_macro namespace="${namespace}" fin_id="5" mesh_filename="${back_down_fin_mesh_file}">
         <origin xyz="-3.44814 0 -0.40858" rpy="${0 * pi} 0 0" />
-    </xacro:aft_fin_macro>
+    </xacro:back_fin_macro>
 </robot>

File: urdf/snippets.xacro (robot description, xacro)
@@ -85,5 +85,5 @@
     <!-- MACRO FOR FIN/RUDDER UNITS  -->
   <!-- A separate mesh for the fin should be stored in the meshes folder -->
-  <xacro:property name="front_left_fin_mesh_file" value="file://$(find O_29qt)/meshes/0.21/front_fin_left_0.21.dae"/>
+  <!--<xacro:property name="front_left_fin_mesh_file" value="file://$(find O_29qt)/meshes/0.21/front_fin_left_0.21.dae"/>
   <xacro:property name="front_right_fin_mesh_file" value="file://$(find O_29qt)/meshes/0.21/front_fin_right_rev_0.21.dae"/>
   <xacro:property name="back_left_fin_mesh_file" value="file://$(find O_29qt)/meshes/0.21/back_fin_left_0.21.dae"/>
@@ -92,5 +92,9 @@
   <xacro:property name="back_down_fin_mesh_file" value="file://$(find O_29qt)/meshes/0.21/back_fin_down_0.21.dae"/>
   <xacro:property name="backup_front_fin_mesh_file" value="file://$(find armsauv_description)/meshes/front_fin.dae"/>
-  <xacro:property name="backup_back_fin_mesh_file" value="file://$(find armsauv_description)/meshes/aft_fin.dae"/>
+  <xacro:property name="backup_back_fin_mesh_file" value="file://$(find armsauv_description)/meshes/aft_fin.dae"/>-->
+  <xacro:property name="front_left_fin_mesh_file" value="file://$(find O_29qt)/meshes/standard/front_left_fin.dae"/>
+  <xacro:property name="front_right_fin_mesh_file" value="file://$(find O_29qt)/meshes/standard/front_right_fin.dae"/>
+  <xacro:property name="back_up_fin_mesh_file" value="file://$(find O_29qt)/meshes/standard/back_up_fin.dae"/>
+  <xacro:property name="back_down_fin_mesh_file" value="file://$(find O_29qt)/meshes/standard/back_down_fin.dae"/>
   <!-- Fin properties -->
   <xacro:property name="fin_rho" value="1025"/>
@@ -132,9 +136,9 @@
   <!--<xacro:property name="aft_fin_area" value="2.656049"/>-->
   <!--<xacro:property name="aft_fin_area" value="0.0172"/>-->
-  <xacro:property name="aft_fin_area" value="0.106243"/>
+  <xacro:property name="back_fin_area" value="0.106243"/>
   <!--<xacro:property name="aft_fin_lift_coefficient" value="3.290443227"/>
   <xacro:property name="aft_fin_drag_coefficient" value="0.269448395"/>-->
-  <xacro:property name="aft_fin_lift_coefficient" value="1.74975211"/>
-  <xacro:property name="aft_fin_drag_coefficient" value="0.269448395"/>
+  <xacro:property name="back_fin_lift_coefficient" value="1.74975211"/>
+  <xacro:property name="back_fin_drag_coefficient" value="0.269448395"/>
   <xacro:macro name="back_left_fin_macro" params="namespace fin_id *origin mesh_filename"> <xacro:hor_left_fin_quadratic_macro
         namespace="${namespace}"
@@ -211,5 +215,5 @@
       </xacro:fin_quadratic_macro>
   </xacro:macro>
-  <xacro:macro name="aft_fin_macro" params="namespace fin_id *origin mesh_filename">
+  <xacro:macro name="back_fin_macro" params="namespace fin_id *origin mesh_filename">
       <xacro:fin_quadratic_macro
         namespace="${namespace}"
@@ -220,6 +224,6 @@
         mesh_filename="${mesh_filename}"
         fin_dynamics_time_constant="0.2"
-        lift_constant="${0.5 * fin_rho * aft_fin_area * aft_fin_lift_coefficient}"
-        drag_constant="${0.5 * fin_rho * aft_fin_area * aft_fin_drag_coefficient}"
+        lift_constant="${0.5 * fin_rho * back_fin_area * back_fin_lift_coefficient}"
+        drag_constant="${0.5 * fin_rho * back_fin_area * back_fin_drag_coefficient}"
         current_velocity_topic="current_velocity">
         <xacro:insert_block name="origin"/>
