Commit message: Update model xacro

File: urdf/actuators_original.xacro (robot description, xacro)
@@ -2,29 +2,27 @@
 <robot xmlns:xacro="http://www.ros.org/wiki/xacro">
     <xacro:thruster_macro robot_namespace="${namespace}" thruster_id = "0">
-        <origin xyz="-20.432 0.0 0.0" rpy="0 0 0" />
+        <origin xyz="-21.77 0.0 0.0" rpy="0 0 0" />
     </xacro:thruster_macro>
-    <xacro:front_fin_macro namespace="${namespace}" fin_id="0" mesh_filename="${front_fin_mesh_file}">
-        <!--<origin xyz="10.2108 -2.3958 -1.3989" rpy="${0.5 * pi} 0 0" />-->
-        <origin xyz="10.2108 -2.3958 0.0" rpy="${0.5 * pi} 0 0" />
-    </xacro:front_fin_macro>
-    <xacro:front_fin_macro namespace="${namespace}" fin_id="1" mesh_filename="${front_fin_mesh_file}">
-        <!--<origin xyz="10.2108 2.3958 -1.3989" rpy="${1.5 * pi} 0 0" />-->
-        <origin xyz="10.2108 2.3958 0.0" rpy="${1.5 * pi} 0 0" />
-    </xacro:front_fin_macro>
-    <xacro:aft_fin_macro namespace="${namespace}" fin_id="2" mesh_filename="${aft_fin_mesh_file}">
-        <!--<origin xyz="-16.583 2.2397 -0.4013" rpy="${0.5 * pi} 0 0" />-->
-        <origin xyz="-16.583 2.2397 0.0" rpy="${0.5 * pi} 0 0" />
-    </xacro:aft_fin_macro>
-    <xacro:aft_fin_macro namespace="${namespace}" fin_id="3" mesh_filename="${aft_fin_mesh_file}">
-        <!--<origin xyz="-16.583 0.0 2.25677" rpy="${1.0 * pi} 0 0" />-->
-        <origin xyz="-16.583 0.0 2.25677" rpy="${1.0 * pi} 0 0" />
-    </xacro:aft_fin_macro>
-    <xacro:aft_fin_macro namespace="${namespace}" fin_id="4" mesh_filename="${aft_fin_mesh_file}">
-        <!--<origin xyz="-16.583 -2.2397 -0.4013" rpy="${1.5 * pi} 0 0" />-->
-        <origin xyz="-16.583 -2.2397 0.0" rpy="${1.5 * pi} 0 0" />
-    </xacro:aft_fin_macro>
-    <xacro:aft_fin_macro namespace="${namespace}" fin_id="5" mesh_filename="${aft_fin_mesh_file}">
-        <!--<origin xyz="-16.583 0.0 -2.25677" rpy="${0.0 * pi} 0 0" />-->
-        <origin xyz="-16.583 0.0 -2.25677" rpy="${0.0 * pi} 0 0" />
-    </xacro:aft_fin_macro>
+    <xacro:front_left_fin_macro namespace="${namespace}" fin_id="0" mesh_filename="${front_left_fin_mesh_file}">
+        <origin xyz="10.411 2.1937 1.20" rpy="0 0 0" />
+        <axiz xyz="0 1 0"/>
+    </xacro:front_left_fin_macro>
+    <xacro:front_right_fin_macro namespace="${namespace}" fin_id="1" mesh_filename="${front_left_fin_mesh_file}">
+        <origin xyz="10.411 -2.1937 1.20" rpy="0 0 0" />
+        <axiz xyz="0 1 0"/>
+    </xacro:front_right_fin_macro>
+    <xacro:front_left_fin_macro namespace="${namespace}" fin_id="2" mesh_filename="${front_left_fin_mesh_file}">
+        <origin xyz="-16.385 2.0 0.395" rpy="0 0 0" />
+        <axiz xyz="0 1 0"/>
+    </xacro:front_left_fin_macro>
+    <xacro:back_up_fin_macro namespace="${namespace}" fin_id="3" mesh_filename="${back_up_fin_mesh_file}">
+        <origin xyz="-16.385 0.0 1.8456" rpy="0 0 0"/>
+    </xacro:back_up_fin_macro>
+    <xacro:front_right_fin_macro namespace="${namespace}" fin_id="4" mesh_filename="${front_left_fin_mesh_file}">
+        <origin xyz="-16.385 -2.0 0.395" rpy="0 0 0" />
+        <axiz xyz="0 1 0"/>
+    </xacro:front_right_fin_macro>
+    <xacro:back_down_fin_macro namespace="${namespace}" fin_id="5" mesh_filename="${back_up_fin_mesh_file}">
+        <origin xyz="-16.385 0.0 -1.8456" rpy="0 0 0"/>
+    </xacro:back_down_fin_macro>
 </robot>

File: urdf/base.xacro (robot description, xacro)
@@ -28,5 +28,5 @@
               <origin rpy="0 0 0" xyz="0 0 0"/>
               <geometry>
-                  <mesh filename="package://O_29qt/meshes/base_link_no_fins.STL"/>
+                  <mesh filename="package://O_29qt/meshes/O_29_base.dae"/>
               </geometry>
               <material name="">
@@ -37,5 +37,5 @@
               <origin rpy="0 0 0" xyz="0 0 0"/>
               <geometry>
-                <mesh filename="package://O_29qt/meshes/base_link_no_fins.STL"/>
+                <mesh filename="package://O_29qt/meshes/O_29_base.dae"/>
               </geometry>
             </collision>

File: urdf/base_original.xacro (robot description, xacro)
@@ -19,10 +19,12 @@
                 <!--<origin rpy="0 0 0" xyz="0 0 0.0086"/>-->
                 <mass value="819026.342183402"/>
-                <inertia ixx="1439809.19440102" ixy="205163.256495052" ixz="-240460.141925145" iyy="24924095.2244092" iyz="-3294.60477684522" izz="25510047.9278752"/>
+                <!--<inertia ixx="1439809.19440102" ixy="205163.256495052" ixz="-240460.141925145" iyy="24924095.2244092" iyz="-3294.60477684522" izz="25510047.9278752"/>-->
+                <inertia ixx="1439809.19440102" ixy="0.0" ixz="0.0" iyy="24924095.2244092" iyz="0.0" izz="25510047.9278752"/>
             </inertial>
             <visual>
               <origin rpy="0 0 0" xyz="0 0 0"/>
               <geometry>
-                  <mesh filename="package://O_29qt/meshes/base_link_ano.STL"/>
+                  <!--<mesh filename="package://O_29qt/meshes/base_link_ano.STL"/>-->
+                  <mesh filename="package://O_29qt/meshes/O_29_base.dae"/>
               </geometry>
               <material name="">
@@ -33,32 +35,9 @@
               <origin rpy="0 0 0" xyz="0 0 0"/>
               <geometry>
-                <mesh filename="package://O_29qt/meshes/base_link_ano.STL"/>
+                  <!--<mesh filename="package://O_29qt/meshes/base_link_ano.STL"/>-->
+                  <mesh filename="package://O_29qt/meshes/O_29_base.dae"/>
               </geometry>
             </collision>
         </link>
-        <!-- <link name="${namespace}/base_link">
-            <inertial>
-              <origin rpy="0 0 0" xyz="4.07474419314708 -0.0300724743266745 -2.34408677014207"/>
-              <mass value="819026.342183402"/>
-              <inertia ixx="1439809.19440102" ixy="205163.256495052" ixz="-240460.141925145" iyy="24924095.2244092" iyz="-3294.60477684522" izz="25510047.9278752"/>
-            </inertial>
-            <visual>
-              <origin rpy="0 0 0" xyz="0 0 0"/>
-              <geometry>
-                  <mesh filename="package://O_29qt/meshes/base_link.STL"/>
-                  <mesh filename="package://O_29qt/meshes/QT1.STL"/>
-                  <mesh filename="package://O_29qt/meshes/base_link_ano.STL"/>
-              </geometry>
-              <material name="">
-                <color rgba="1 0.0588235294117647 0.458823529411765 1"/>
-              </material>
-            </visual>
-            <collision>
-              <origin rpy="0 0 0" xyz="0 0 0"/>
-              <geometry>
-                <mesh filename="package://O_29qt/meshes/base_link.STL"/>
-              </geometry>
-            </collision>
-        </link>-->
         <gazebo reference="${namespace}/base_link">
             <selfCollide>false</selfCollide>
@@ -68,5 +47,5 @@
         <xacro:include filename="$(find O_29qt)/urdf/actuators_original.xacro"/>
         <!-- Include the sensor modules -->
-        <xacro:include filename="$(find O_29qt)/urdf/sensors.xacro"/>
+        <xacro:include filename="$(find O_29qt)/urdf/sensors_original.xacro"/>
     </xacro:macro>
 </robot>

File: urdf/gazebo.xacro (robot description, xacro)
@@ -20,7 +20,7 @@
     <!-- Added base parameters -->
     <xacro:property name="O_29qt_length" value="8.534"/>
-    <xacro:property name="O_29qt_width"  value="2.94525"/>
+    <xacro:property name="O_29qt_width"  value="1.0256"/>
     <xacro:property name="O_29qt_radius"  value="0.5128"/>
-    <xacro:property name="O_29qt_height" value="1.5246"/>
+    <xacro:property name="O_29qt_height" value="1.0256"/>
     <xacro:property name="rho" value="1025" />
     <xacro:property name="D0" value="${rho * 0.5}"/>

File: urdf/snippets.xacro (robot description, xacro)
@@ -85,8 +85,8 @@
     <!-- MACRO FOR FIN/RUDDER UNITS  -->
   <!-- A separate mesh for the fin should be stored in the meshes folder -->
-  <!--<xacro:property name="front_fin_mesh_file" value="file://$(find O_29qt)/meshes/front_fin_latest.STL"/>-->
-  <xacro:property name="front_fin_mesh_file" value="file://$(find armsauv_description)/meshes/front_fin.dae"/>
-  <!--<xacro:property name="aft_fin_mesh_file" value="file://$(find O_29qt)/meshes/aft_fin_latest.STL"/>-->
-  <xacro:property name="aft_fin_mesh_file" value="file://$(find armsauv_description)/meshes/aft_fin.dae"/>
+  <xacro:property name="front_fin_mesh_file" value="file://$(find O_29qt)/meshes/front_fin_latest.STL"/>
+  <!--<xacro:property name="front_fin_mesh_file" value="file://$(find armsauv_description)/meshes/front_fin.dae"/>-->
+  <xacro:property name="aft_fin_mesh_file" value="file://$(find O_29qt)/meshes/aft_fin_latest.STL"/>
+  <!--<xacro:property name="aft_fin_mesh_file" value="file://$(find armsauv_description)/meshes/aft_fin.dae"/>-->
   <!-- Fin properties -->
   <xacro:property name="fin_rho" value="1025"/>
@@ -98,5 +98,5 @@
   <xacro:property name="front_fin_drag_coefficient" value="0.26542681"/>
   <xacro:macro name="front_fin_macro" params="namespace fin_id *origin mesh_filename">
-      <xacro:fin_quadratic_macro
+      <!--<xacro:fin_quadratic_macro
         namespace="${namespace}"
         parent_link="${namespace}/base_link" fin_id="${fin_id}"
@@ -109,15 +109,16 @@
         current_velocity_topic="current_velocity">
         <xacro:insert_block name="origin"/>
-      </xacro:fin_quadratic_macro>
-      <!--<link name="${namespace}/fin${fin_id}">
+      </xacro:fin_quadratic_macro>-->
+      <link name="${namespace}/fin${fin_id}">
+          <xacro:no_inertial/>
           <visual>
               <origin xyz="0 0 0" rpy="0 0 0"/>
               <geometry>
-                  <mesh filename="${mesh_filename}" scale="9 9 9"/>
+                  <mesh filename="${mesh_filename}" scale="1 1 1"/>
               </geometry>
           </visual>
       </link>
       <joint name="${namespace}/fin${fin_id}_joint" type="revolute">
-          <limit effort="0" lower="${-30*d2r}" upper="${30*d2r}" velocity="0"/>
+          <limit effort="0" lower="${-90*d2r}" upper="${90*d2r}" velocity="0"/>
           <xacro:insert_block name="origin"/>
           <axiz xyz="0 0 1"/>
@@ -129,5 +130,5 @@
               <dynamics>
                   <type>FirstOrder</type>
-                  <timeConstant>0.1</timeConstant>
+                  <timeConstant>0.2</timeConstant>
               </dynamics>
               <liftdrag>
@@ -141,5 +142,5 @@
               <joint_name>${namespace}/fin${fin_id}_joint</joint_name>
           </plugin>
-      </gazebo>-->
+      </gazebo>
   </xacro:macro>
   <!--<xacro:property name="aft_fin_area" value="2.656049"/>-->
@@ -150,5 +151,5 @@
   <xacro:property name="aft_fin_drag_coefficient" value="0.269448395"/>
   <xacro:macro name="aft_fin_macro" params="namespace fin_id *origin mesh_filename">
-      <xacro:fin_quadratic_macro
+      <!--<xacro:fin_quadratic_macro
         namespace="${namespace}"
         parent_link="${namespace}/base_link"
@@ -162,5 +163,38 @@
         current_velocity_topic="current_velocity">
         <xacro:insert_block name="origin"/>
-      </xacro:fin_quadratic_macro>
+      </xacro:fin_quadratic_macro>-->
+      <link name="${namespace}/fin${fin_id}">
+          <xacro:no_inertial/>
+          <visual>
+              <origin xyz="0 0 0" rpy="0 0 0"/>
+              <geometry>
+                  <mesh filename="${mesh_filename}" scale="1 1 1"/>
+              </geometry>
+          </visual>
+      </link>
+      <joint name="${namespace}/fin${fin_id}_joint" type="revolute">
+          <limit effort="0" lower="${-90*d2r}" upper="${90*d2r}" velocity="0"/>
+          <xacro:insert_block name="origin"/>
+          <axiz xyz="0 0 1"/>
+          <parent link="${namespace}/base_link"/>
+          <child link="${namespace}/fin${fin_id}"/>
+      </joint>
+      <gazebo>
+          <plugin name="${namespace}_fin${fin_id}_model" filename="libuuv_fin_ros_plugin.so">
+              <dynamics>
+                  <type>FirstOrder</type>
+                  <timeConstant>0.2</timeConstant>
+              </dynamics>
+              <liftdrag>
+                  <type>Quadratic</type>
+                  <lift_constant>${0.5 * fin_rho * front_fin_area * front_fin_lift_coefficient}</lift_constant>
+                  <drag_constant>${0.5 * fin_rho * front_fin_area * front_fin_drag_coefficient}</drag_constant>
+              </liftdrag>
+              <current_velocity_topic>current_velocity</current_velocity_topic>
+              <fin_id>${fin_id}</fin_id>
+              <link_name>${namespace}/fin${fin_id}</link_name>
+              <joint_name>${namespace}/fin${fin_id}_joint</joint_name>
+          </plugin>
+      </gazebo>
   </xacro:macro>
   <!-- <xacro:macro name="fin_macro" params="namespace fin_id *origin mesh_filename">
