Commit message: Update model xacro

File: urdf/snippets_original.xacro (robot description, xacro)
@@ -1,5 +1,5 @@
 <?xml version="1.0" encoding="UTF-8"?>
 <robot xmlns:xacro="http://www.ros.org/wiki/xacro">
-    <xacro:property name="propeller_mesh_file" value="file://$(find O_29qt)/meshes/propeller.STL" />
+    <xacro:property name="propeller_mesh_file" value="file://$(find O_29qt)/meshes/propeller.dae" />
     <xacro:macro name="thruster_macro" params="robot_namespace thruster_id *origin">
         <link name="${robot_namespace}/thruster_${thruster_id}">
@@ -85,6 +85,9 @@
     <!-- MACRO FOR FIN/RUDDER UNITS  -->
   <!-- A separate mesh for the fin should be stored in the meshes folder -->
-  <xacro:property name="front_fin_mesh_file" value="file://$(find O_29qt)/meshes/front_fin.dae"/>
-  <xacro:property name="aft_fin_mesh_file" value="file://$(find O_29qt)/meshes/aft_fin.dae"/>
+  <!--<xacro:property name="front_fin_mesh_file" value="file://$(find O_29qt)/meshes/front_fin_latest.STL"/>-->
+  <!--<xacro:property name="aft_fin_mesh_file" value="file://$(find O_29qt)/meshes/aft_fin_latest.STL"/>-->
+  <xacro:property name="front_left_fin_mesh_file" value="file://$(find O_29qt)/meshes/front_fin_left_new.dae"/>
+  <!--<xacro:property name="front_left_fin_mesh_file" value="file://$(find O_29qt)/meshes/horizontal_fin.dae"/>-->
+  <xacro:property name="back_up_fin_mesh_file" value="file://$(find O_29qt)/meshes/back_fin_up_new.dae"/>
   <!-- Fin properties -->
   <xacro:property name="fin_rho" value="1025"/>
@@ -93,17 +96,73 @@
   <xacro:property name="front_fin_lift_coefficient" value="20.843"/>
   <xacro:property name="front_fin_drag_coefficient" value="1.98"/>
-  <xacro:macro name="front_fin_macro" params="namespace fin_id *origin mesh_filename">
-      <xacro:fin_quadratic_macro
-        namespace="${namespace}"
-        parent_link="${namespace}/base_link" fin_id="${fin_id}"
-        min_joint_limit="${-90.0 * d2r}"
-        max_joint_limit="${90.0 * d2r}"
-        mesh_filename="${mesh_filename}"
-        fin_dynamics_time_constant="0.2"
-        lift_constant="${0.5 * fin_rho * front_fin_area * front_fin_lift_coefficient}"
-        drag_constant="${0.5 * fin_rho * front_fin_area * front_fin_drag_coefficient}"
-        current_velocity_topic="current_velocity">
-        <xacro:insert_block name="origin"/>
-      </xacro:fin_quadratic_macro>
+  <xacro:macro name="front_left_fin_macro" params="namespace fin_id *origin *axiz mesh_filename">
+    <link name="${namespace}/fin${fin_id}">
+      <xacro:no_inertial/>
+      <visual>
+          <origin xyz="0 0 0" rpy="0 0 0"/>
+          <geometry>
+              <mesh filename="${mesh_filename}" scale="1 1 1"/>
+          </geometry>
+      </visual>
+    </link>
+    <joint name="${namespace}/fin${fin_id}_joint" type="revolute">
+      <limit effort="0" lower="${-90*d2r}" upper="${90*d2r}" velocity="0"/>
+      <xacro:insert_block name="origin"/>
+      <xacro:insert_block name="axiz"/>
+      <parent link="${namespace}/base_link"/>
+      <child link="${namespace}/fin${fin_id}"/>
+    </joint>
+    <gazebo>
+      <plugin name="${namespace}_fin${fin_id}_model" filename="libuuv_fin_ros_plugin.so">
+          <dynamics>
+              <type>FirstOrder</type>
+              <timeConstant>0.2</timeConstant>
+          </dynamics>
+          <liftdrag>
+              <type>Quadratic</type>
+              <lift_constant>${0.5 * fin_rho * front_fin_area * front_fin_lift_coefficient}</lift_constant>
+              <drag_constant>${0.5 * fin_rho * front_fin_area * front_fin_drag_coefficient}</drag_constant>
+          </liftdrag>
+          <current_velocity_topic>current_velocity</current_velocity_topic>
+          <fin_id>${fin_id}</fin_id>
+          <link_name>${namespace}/fin${fin_id}</link_name>
+          <joint_name>${namespace}/fin${fin_id}_joint</joint_name>
+      </plugin>
+    </gazebo>
+  </xacro:macro>
+  <xacro:macro name="front_right_fin_macro" params="namespace fin_id *origin *axiz mesh_filename">
+    <joint name="${namespace}/fin${fin_id}_joint" type="revolute">
+      <limit effort="0" lower="${-90*d2r}" upper="${90*d2r}" velocity="0"/>
+      <xacro:insert_block name="origin"/>
+      <xacro:insert_block name="axiz"/>
+      <parent link="${namespace}/base_link"/>
+      <child link="${namespace}/fin${fin_id}"/>
+    </joint>
+    <link name="${namespace}/fin${fin_id}">
+      <xacro:no_inertial/>
+      <visual>
+          <origin xyz="0 0 0" rpy="0 0 0"/>
+          <geometry>
+              <mesh filename="${mesh_filename}" scale="1 -1 1"/>
+          </geometry>
+      </visual>
+    </link>
+    <gazebo>
+      <plugin name="${namespace}_fin${fin_id}_model" filename="libuuv_fin_ros_plugin.so">
+          <dynamics>
+              <type>FirstOrder</type>
+              <timeConstant>0.2</timeConstant>
+          </dynamics>
+          <liftdrag>
+              <type>Quadratic</type>
+              <lift_constant>${0.5 * fin_rho * front_fin_area * front_fin_lift_coefficient}</lift_constant>
+              <drag_constant>${0.5 * fin_rho * front_fin_area * front_fin_drag_coefficient}</drag_constant>
+          </liftdrag>
+          <current_velocity_topic>current_velocity</current_velocity_topic>
+          <fin_id>${fin_id}</fin_id>
+          <link_name>${namespace}/fin${fin_id}</link_name>
+          <joint_name>${namespace}/fin${fin_id}_joint</joint_name>
+      </plugin>
+    </gazebo>
   </xacro:macro>
   <xacro:property name="aft_fin_area" value="2.656049"/>
@@ -111,62 +170,73 @@
   <xacro:property name="aft_fin_lift_coefficient" value="19.1395"/>
   <xacro:property name="aft_fin_drag_coefficient" value="1.98"/>
-  <xacro:macro name="aft_fin_macro" params="namespace fin_id *origin mesh_filename">
-      <xacro:fin_quadratic_macro
-        namespace="${namespace}"
-        parent_link="${namespace}/base_link"
-        fin_id="${fin_id}"
-        min_joint_limit="${-90.0 * d2r}"
-        max_joint_limit="${90.0 * d2r}"
-        mesh_filename="${mesh_filename}"
-        fin_dynamics_time_constant="0.2"
-        lift_constant="${0.5 * fin_rho * aft_fin_area * aft_fin_lift_coefficient}"
-        drag_constant="${0.5 * fin_rho * aft_fin_area * aft_fin_drag_coefficient}"
-        current_velocity_topic="current_velocity">
-        <xacro:insert_block name="origin"/>
-      </xacro:fin_quadratic_macro>
-  </xacro:macro>
-  <!-- <xacro:macro name="fin_macro" params="namespace fin_id *origin mesh_filename">
-      <xacro:fin_two_lines_macro
-        namespace="${namespace}"
-        parent_link="${namespace}/base_link"
-        fin_id="${fin_id}"
-        min_joint_limit="${-80*d2r}"
-        max_joint_limit="${80*d2r}"
-        mesh_filename="${mesh_filename}"
-        fin_dynamics_time_constant="0.1"
-        fin_cross_section_area="${fin_area}"
-        current_velocity_topic="current_velocity"
-        fluid_density="1025.0"
-        a0="0.0"
-        alpha_stall="1.57"
-        cla="${0.5 * fin_rho * fin_area * fin_lift_coefficient}"
-        cla_stall="0.0"
-        cda="${0.5 * fin_rho * fin_area * fin_drag_coefficient}"
-        cda_stall="0">
-        <xacro:insert_block name="origin"/>
-      </xacro:fin_two_lines_macro>
-    </xacro:macro> -->
-    <!-- <xacro:macro name="fin_macro" params="namespace fin_id *origin mesh_filename">
-      <xacro:fin_two_lines_macro
-        namespace="${namespace}"
-        parent_link="${namespace}/base_link"
-        fin_id="${fin_id}"
-        min_joint_limit="${-80*d2r}"
-        max_joint_limit="${80*d2r}"
-        mesh_filename="${mesh_filename}"
-        fin_dynamics_time_constant="0.1"
-        fin_cross_section_area="${fin_area}"
-        current_velocity_topic="current_velocity"
-        fluid_density="1025.0"
-        a0="0.0"
-        alpha_stall="0.436332313"
-        cla="2.435070629"
-        cla_stall="0"
-        cda="0"
-        cda_stall="0">
-        <xacro:insert_block name="origin"/>
-      </xacro:fin_two_lines_macro>
-    </xacro:macro> -->
-    <!-- cla_stall="-1.929963096"
-        cda="1.101841914" -->
+  <xacro:macro name="back_up_fin_macro" params="namespace fin_id *origin mesh_filename">
+    <link name="${namespace}/fin${fin_id}">
+      <xacro:no_inertial/>
+      <visual>
+          <origin xyz="0 0 0" rpy="0 0 0"/>
+          <geometry>
+              <mesh filename="${mesh_filename}" scale="1 1 1"/>
+          </geometry>
+      </visual>
+    </link>
+    <joint name="${namespace}/fin${fin_id}_joint" type="revolute">
+      <limit effort="0" lower="${-90*d2r}" upper="${90*d2r}" velocity="0"/>
+      <xacro:insert_block name="origin"/>
+      <axiz xyz="0 0 1"/>
+      <parent link="${namespace}/base_link"/>
+      <child link="${namespace}/fin${fin_id}"/>
+    </joint>
+    <gazebo>
+      <plugin name="${namespace}_fin${fin_id}_model" filename="libuuv_fin_ros_plugin.so">
+          <dynamics>
+              <type>FirstOrder</type>
+              <timeConstant>0.2</timeConstant>
+          </dynamics>
+          <liftdrag>
+              <type>Quadratic</type>
+              <lift_constant>${0.5 * fin_rho * aft_fin_area * aft_fin_lift_coefficient}</lift_constant>
+              <drag_constant>${0.5 * fin_rho * aft_fin_area * aft_fin_drag_coefficient}</drag_constant>
+          </liftdrag>
+          <current_velocity_topic>current_velocity</current_velocity_topic>
+          <fin_id>${fin_id}</fin_id>
+          <link_name>${namespace}/fin${fin_id}</link_name>
+          <joint_name>${namespace}/fin${fin_id}_joint</joint_name>
+      </plugin>
+    </gazebo>
+  </xacro:macro>
+  <xacro:macro name="back_down_fin_macro" params="namespace fin_id *origin mesh_filename">
+    <link name="${namespace}/fin${fin_id}">
+      <xacro:no_inertial/>
+      <visual>
+          <origin xyz="0 0 0" rpy="0 0 0"/>
+          <geometry>
+              <mesh filename="${mesh_filename}" scale="1 1 -1"/>
+          </geometry>
+      </visual>
+    </link>
+    <joint name="${namespace}/fin${fin_id}_joint" type="revolute">
+      <limit effort="0" lower="${-90*d2r}" upper="${90*d2r}" velocity="0"/>
+      <xacro:insert_block name="origin"/>
+      <axiz xyz="0 0 1"/>
+      <parent link="${namespace}/base_link"/>
+      <child link="${namespace}/fin${fin_id}"/>
+    </joint>
+    <gazebo>
+      <plugin name="${namespace}_fin${fin_id}_model" filename="libuuv_fin_ros_plugin.so">
+          <dynamics>
+              <type>FirstOrder</type>
+              <timeConstant>0.2</timeConstant>
+          </dynamics>
+          <liftdrag>
+              <type>Quadratic</type>
+              <lift_constant>${0.5 * fin_rho * aft_fin_area * aft_fin_lift_coefficient}</lift_constant>
+              <drag_constant>${0.5 * fin_rho * aft_fin_area * aft_fin_drag_coefficient}</drag_constant>
+          </liftdrag>
+          <current_velocity_topic>current_velocity</current_velocity_topic>
+          <fin_id>${fin_id}</fin_id>
+          <link_name>${namespace}/fin${fin_id}</link_name>
+          <joint_name>${namespace}/fin${fin_id}_joint</joint_name>
+      </plugin>
+    </gazebo>
+  </xacro:macro>
 </robot>

Commit message: Try to solve problems with fin xacro

File: urdf/actuators_original.xacro (robot description, xacro)
@@ -6,13 +6,13 @@
     <xacro:front_left_fin_macro namespace="${namespace}" fin_id="0" mesh_filename="${front_left_fin_mesh_file}">
         <origin xyz="10.411 2.1937 1.20" rpy="0 0 0" />
-        <axiz xyz="0 1 0"/>
+        <axiz xyz="0 0 1"/>
     </xacro:front_left_fin_macro>
     <xacro:front_right_fin_macro namespace="${namespace}" fin_id="1" mesh_filename="${front_left_fin_mesh_file}">
         <origin xyz="10.411 -2.1937 1.20" rpy="0 0 0" />
-        <axiz xyz="0 1 0"/>
+        <axiz xyz="0 0 1"/>
     </xacro:front_right_fin_macro>
     <xacro:front_left_fin_macro namespace="${namespace}" fin_id="2" mesh_filename="${front_left_fin_mesh_file}">
         <origin xyz="-16.385 2.0 0.395" rpy="0 0 0" />
-        <axiz xyz="0 1 0"/>
+        <axiz xyz="0 0 1"/>
     </xacro:front_left_fin_macro>
     <xacro:back_up_fin_macro namespace="${namespace}" fin_id="3" mesh_filename="${back_up_fin_mesh_file}">
@@ -21,5 +21,5 @@
     <xacro:front_right_fin_macro namespace="${namespace}" fin_id="4" mesh_filename="${front_left_fin_mesh_file}">
         <origin xyz="-16.385 -2.0 0.395" rpy="0 0 0" />
-        <axiz xyz="0 1 0"/>
+        <axiz xyz="0 0 1"/>
     </xacro:front_right_fin_macro>
     <xacro:back_down_fin_macro namespace="${namespace}" fin_id="5" mesh_filename="${back_up_fin_mesh_file}">

File: urdf/base_original.xacro (robot description, xacro)
@@ -26,9 +26,9 @@
               <geometry>
                   <!--<mesh filename="package://O_29qt/meshes/base_link_ano.STL"/>-->
-                  <mesh filename="package://O_29qt/meshes/O_29_base.dae"/>
+                  <mesh filename="package://O_29qt/meshes/O_29_base.dae" scale="1 1 1"/>
               </geometry>
-              <material name="">
+              <!--<material name="">
                 <color rgba="1 0.0588235294117647 0.458823529411765 1"/>
-              </material>
+              </material>-->
             </visual>
             <collision>
@@ -36,5 +36,5 @@
               <geometry>
                   <!--<mesh filename="package://O_29qt/meshes/base_link_ano.STL"/>-->
-                  <mesh filename="package://O_29qt/meshes/O_29_base.dae"/>
+                  <mesh filename="package://O_29qt/meshes/O_29_base.dae" scale="1 1 1"/>
               </geometry>
             </collision>

File: urdf/snippets_original.xacro (robot description, xacro)
@@ -85,8 +85,5 @@
     <!-- MACRO FOR FIN/RUDDER UNITS  -->
   <!-- A separate mesh for the fin should be stored in the meshes folder -->
-  <!--<xacro:property name="front_fin_mesh_file" value="file://$(find O_29qt)/meshes/front_fin_latest.STL"/>-->
-  <!--<xacro:property name="aft_fin_mesh_file" value="file://$(find O_29qt)/meshes/aft_fin_latest.STL"/>-->
   <xacro:property name="front_left_fin_mesh_file" value="file://$(find O_29qt)/meshes/front_fin_left_new.dae"/>
-  <!--<xacro:property name="front_left_fin_mesh_file" value="file://$(find O_29qt)/meshes/horizontal_fin.dae"/>-->
   <xacro:property name="back_up_fin_mesh_file" value="file://$(find O_29qt)/meshes/back_fin_up_new.dae"/>
   <!-- Fin properties -->
@@ -98,5 +95,5 @@
   <xacro:macro name="front_left_fin_macro" params="namespace fin_id *origin *axiz mesh_filename">
     <link name="${namespace}/fin${fin_id}">
-      <xacro:no_inertial/>
+      <!--<xacro:no_inertial/>-->
       <visual>
           <origin xyz="0 0 0" rpy="0 0 0"/>
@@ -105,4 +102,9 @@
           </geometry>
       </visual>
+      <inertial>
+          <mass value="0.001" />
+          <origin xyz="0 0 0" rpy="0 0 0" />
+          <inertia ixx="0.000000001" ixy="0.0" ixz="0.0" iyy="0.000000001" iyz="0.0" izz="0.000000001" />
+      </inertial>
     </link>
     <joint name="${namespace}/fin${fin_id}_joint" type="revolute">
@@ -140,5 +142,5 @@
     </joint>
     <link name="${namespace}/fin${fin_id}">
-      <xacro:no_inertial/>
+      <!--<xacro:no_inertial/>-->
       <visual>
           <origin xyz="0 0 0" rpy="0 0 0"/>
@@ -147,4 +149,11 @@
           </geometry>
       </visual>
+      <inertial>
+          <mass value="0.001" />
+          <origin xyz="0 0 0" rpy="0 0 0" />
+          <inertia ixx="0.000000001" ixy="0.0" ixz="0.0"
+              iyy="0.000000001" iyz="0.0"
+              izz="0.000000001" />
+      </inertial>
     </link>
     <gazebo>
@@ -172,5 +181,5 @@
   <xacro:macro name="back_up_fin_macro" params="namespace fin_id *origin mesh_filename">
     <link name="${namespace}/fin${fin_id}">
-      <xacro:no_inertial/>
+      <!--<xacro:no_inertial/>-->
       <visual>
           <origin xyz="0 0 0" rpy="0 0 0"/>
@@ -179,4 +188,9 @@
           </geometry>
       </visual>
+      <inertial>
+          <mass value="0.001" />
+          <origin xyz="0 0 0" rpy="0 0 0" />
+          <inertia ixx="0.000000001" ixy="0.0" ixz="0.0" iyy="0.000000001" iyz="0.0" izz="0.000000001" />
+      </inertial>
     </link>
     <joint name="${namespace}/fin${fin_id}_joint" type="revolute">
@@ -207,5 +221,5 @@
   <xacro:macro name="back_down_fin_macro" params="namespace fin_id *origin mesh_filename">
     <link name="${namespace}/fin${fin_id}">
-      <xacro:no_inertial/>
+      <!--<xacro:no_inertial/>-->
       <visual>
           <origin xyz="0 0 0" rpy="0 0 0"/>
@@ -214,4 +228,9 @@
           </geometry>
       </visual>
+      <inertial>
+          <mass value="0.001" />
+          <origin xyz="0 0 0" rpy="0 0 0" />
+          <inertia ixx="0.000000001" ixy="0.0" ixz="0.0" iyy="0.000000001" iyz="0.0" izz="0.000000001" />
+      </inertial>
     </link>
     <joint name="${namespace}/fin${fin_id}_joint" type="revolute">
