Commit message: Modify model xacros

File: urdf/actuators_original.xacro (robot description, xacro)
@@ -6,22 +6,19 @@
     <xacro:front_left_fin_macro namespace="${namespace}" fin_id="0" mesh_filename="${front_left_fin_mesh_file}">
         <origin xyz="10.411 2.1937 1.20" rpy="0 0 0" />
-        <axiz xyz="0 0 1"/>
     </xacro:front_left_fin_macro>
-    <xacro:front_right_fin_macro namespace="${namespace}" fin_id="1" mesh_filename="${front_left_fin_mesh_file}">
+    <!--<xacro:front_right_fin_macro namespace="${namespace}" fin_id="1" mesh_filename="${front_left_fin_mesh_file}">-->
+    <xacro:front_right_fin_macro namespace="${namespace}" fin_id="1" mesh_filename="${front_right_fin_mesh_file}">
         <origin xyz="10.411 -2.1937 1.20" rpy="0 0 0" />
-        <axiz xyz="0 0 1"/>
     </xacro:front_right_fin_macro>
     <xacro:front_left_fin_macro namespace="${namespace}" fin_id="2" mesh_filename="${front_left_fin_mesh_file}">
         <origin xyz="-16.385 2.0 0.395" rpy="0 0 0" />
-        <axiz xyz="0 0 1"/>
     </xacro:front_left_fin_macro>
     <xacro:back_up_fin_macro namespace="${namespace}" fin_id="3" mesh_filename="${back_up_fin_mesh_file}">
         <origin xyz="-16.385 0.0 1.8456" rpy="0 0 0"/>
     </xacro:back_up_fin_macro>
-    <xacro:front_right_fin_macro namespace="${namespace}" fin_id="4" mesh_filename="${front_left_fin_mesh_file}">
+    <xacro:front_right_fin_macro namespace="${namespace}" fin_id="4" mesh_filename="${front_right_fin_mesh_file}">
         <origin xyz="-16.385 -2.0 0.395" rpy="0 0 0" />
-        <axiz xyz="0 0 1"/>
     </xacro:front_right_fin_macro>
-    <xacro:back_down_fin_macro namespace="${namespace}" fin_id="5" mesh_filename="${back_up_fin_mesh_file}">
+    <xacro:back_down_fin_macro namespace="${namespace}" fin_id="5" mesh_filename="${back_down_fin_mesh_file}">
         <origin xyz="-16.385 0.0 -1.8456" rpy="0 0 0"/>
     </xacro:back_down_fin_macro>

File: urdf/base_original.xacro (robot description, xacro)
@@ -17,5 +17,4 @@
             <inertial>
                 <origin rpy="0 0 0" xyz="0 0 0"/>
-                <!--<origin rpy="0 0 0" xyz="0 0 0.0086"/>-->
                 <mass value="819026.342183402"/>
                 <!--<inertia ixx="1439809.19440102" ixy="205163.256495052" ixz="-240460.141925145" iyy="24924095.2244092" iyz="-3294.60477684522" izz="25510047.9278752"/>-->
@@ -25,6 +24,6 @@
               <origin rpy="0 0 0" xyz="0 0 0"/>
               <geometry>
-                  <!--<mesh filename="package://O_29qt/meshes/base_link_ano.STL"/>-->
-                  <mesh filename="package://O_29qt/meshes/O_29_base.dae" scale="1 1 1"/>
+                  <!--<mesh filename="package://O_29qt/meshes/base_link_ano.STL" scale="1 1 1"/>-->
+                  <mesh filename="file://$(find O_29qt)/meshes/O_29_base.dae" scale="1 1 1"/>
               </geometry>
               <!--<material name="">
@@ -35,6 +34,6 @@
               <origin rpy="0 0 0" xyz="0 0 0"/>
               <geometry>
-                  <!--<mesh filename="package://O_29qt/meshes/base_link_ano.STL"/>-->
-                  <mesh filename="package://O_29qt/meshes/O_29_base.dae" scale="1 1 1"/>
+                  <!--<mesh filename="package://O_29qt/meshes/base_link_ano.STL" scale="1 1 1"/>-->
+                  <mesh filename="file://$(find O_29qt)/meshes/O_29_base.dae" scale="1 1 1"/>
               </geometry>
             </collision>

File: urdf/gazebo.xacro (robot description, xacro)
@@ -4,18 +4,6 @@
     <xacro:property name="O_29qt_cob" value="0 0 0"/>
     <!-- Vehicle's actual volume (Gazebo cannot compute the volume out of the mesh) -->
-    <!--<xacro:property name="O_29qt_volume" value="${819026 / 9.8 / 1000}"/>-->
-    <!--<xacro:property name="O_29qt_volume" value="${838 / 9.8 / 1000}"/>-->
     <!--<xacro:property name="O_29qt_volume" value="${4690 / 1000}"/>-->
     <xacro:property name="O_29qt_volume" value="${4390 / 1000}"/>
-    <!-- Describing the dimensions of the vehicle's bounding box -->
-    <!--<xacro:property name="O_29qt_length" value="40.97"/>
-    <xacro:property name="O_29qt_width"  value="4.923"/>
-    <xacro:property name="O_29qt_radius"  value="2.4615"/>
-    <xacro:property name="O_29qt_height" value="4.923"/>-->
-    <!-- Added base parameters(ARMSAUA) -->
-    <!--<xacro:property name="O_29qt_length" value="2.712"/>
-    <xacro:property name="O_29qt_width"  value="0.935"/>
-    <xacro:property name="O_29qt_radius"  value="0.120"/>
-    <xacro:property name="O_29qt_height" value="0.484"/>-->
     <!-- Added base parameters -->
     <xacro:property name="O_29qt_length" value="8.534"/>

File: urdf/gazebo_original.xacro (robot description, xacro)
@@ -3,4 +3,5 @@
     <!-- Center of buoyancy -->
     <xacro:property name="O_29qt_cob" value="0 0 0"/>
+    <!--<xacro:property name="O_29qt_cob" value="0.4129 0 -0.6577"/>-->
     <!-- Vehicle's actual volume (Gazebo cannot compute the volume out of the mesh) -->
     <xacro:property name="O_29qt_volume" value="${819026 / 1000}"/>

File: urdf/snippets_original.xacro (robot description, xacro)
@@ -35,11 +35,11 @@
                 <gain>1</gain>
                 <!-- Maximum allowed input value for the input signal for thruster unit -->
-                <clampMax>2300</clampMax>
+                <clampMax>2500</clampMax>
                 <!-- Minimum allowed input value for the input signal for thruster unit -->
-                <clampMin>-2300</clampMin>
+                <clampMin>-2500</clampMin>
                 <!-- Maximum thrust force output allowed -->
-                <thrustMax>26338.811</thrustMax>
+                <thrustMax>263388.11</thrustMax>
                 <!-- Minimum thrust force output allowed -->
-                <thrustMin>-26338.811</thrustMin>
+                <thrustMin>-263388.11</thrustMin>
                 <!--
                 Value from 0 to 1 to set the efficiency of the output thrus
@@ -75,5 +75,5 @@
                     <type>LinearInterp</type>
                     <inputValues>0 500 1000 1500 2000 2500</inputValues>
-                    <outputValues>0 1053.5524 4214.2097 9481.9719 16856.839 26338.811</outputValues>
+                    <outputValues>0 10535.524 42142.097 94819.719 168568.39 263388.11</outputValues>
                 </conversion>
             </plugin>
@@ -86,14 +86,27 @@
   <!-- A separate mesh for the fin should be stored in the meshes folder -->
   <xacro:property name="front_left_fin_mesh_file" value="file://$(find O_29qt)/meshes/front_fin_left_new.dae"/>
+  <xacro:property name="front_right_fin_mesh_file" value="file://$(find O_29qt)/meshes/front_fin_right_new.dae"/>
   <xacro:property name="back_up_fin_mesh_file" value="file://$(find O_29qt)/meshes/back_fin_up_new.dae"/>
+  <xacro:property name="back_down_fin_mesh_file" value="file://$(find O_29qt)/meshes/back_fin_down_new.dae"/>
   <!-- Fin properties -->
   <xacro:property name="fin_rho" value="1025"/>
   <xacro:property name="front_fin_area" value="2.9153726"/>
-  <!--<xacro:property name="front_fin_area" value="0.785"/>-->
-  <xacro:property name="front_fin_lift_coefficient" value="20.843"/>
-  <xacro:property name="front_fin_drag_coefficient" value="1.98"/>
-  <xacro:macro name="front_left_fin_macro" params="namespace fin_id *origin *axiz mesh_filename">
-    <link name="${namespace}/fin${fin_id}">
-      <!--<xacro:no_inertial/>-->
+  <xacro:property name="front_fin_lift_coefficient" value="1.668475641"/>
+  <xacro:property name="front_fin_drag_coefficient" value="0.26542681"/>
+  <xacro:macro name="front_left_fin_macro" params="namespace fin_id *origin mesh_filename">
+    <xacro:hor_left_fin_quadratic_macro
+        namespace="${namespace}"
+        parent_link="${namespace}/base_link"
+        fin_id="${fin_id}"
+        min_joint_limit="${-90.0*d2r}"
+        max_joint_limit="${90.0*d2r}"
+        mesh_filename="${mesh_filename}"
+        fin_dynamics_time_constant="0.2"
+        lift_constant="${0.5 * fin_rho * front_fin_area * front_fin_lift_coefficient}"
+        drag_constant="${0.5 * fin_rho * front_fin_area * front_fin_drag_coefficient}"
+        current_velocity_topic="current_velocity">
+        <xacro:insert_block name="origin"/>
+    </xacro:hor_left_fin_quadratic_macro>
+    <!--<link name="${namespace}/fin${fin_id}">
       <visual>
           <origin xyz="0 0 0" rpy="0 0 0"/>
@@ -131,7 +144,22 @@
           <joint_name>${namespace}/fin${fin_id}_joint</joint_name>
       </plugin>
-    </gazebo>
+    </gazebo>-->
   </xacro:macro>
-  <xacro:macro name="front_right_fin_macro" params="namespace fin_id *origin *axiz mesh_filename">
+  <xacro:macro name="front_right_fin_macro" params="namespace fin_id *origin mesh_filename">
+    <xacro:hor_right_fin_quadratic_macro
+        namespace="${namespace}"
+        parent_link="${namespace}/base_link"
+        fin_id="${fin_id}"
+        min_joint_limit="${-90.0*d2r}"
+        max_joint_limit="${90.0*d2r}"
+        mesh_filename="${mesh_filename}"
+        fin_dynamics_time_constant="0.2"
+        lift_constant="${0.5 * fin_rho * front_fin_area * front_fin_lift_coefficient}"
+        drag_constant="${0.5 * fin_rho * front_fin_area * front_fin_drag_coefficient}"
+        current_velocity_topic="current_velocity">
+        <xacro:insert_block name="origin"/>
+    </xacro:hor_right_fin_quadratic_macro>
+    <!--<link name="${namespace}/fin${fin_id}">
+      <visual>
     <joint name="${namespace}/fin${fin_id}_joint" type="revolute">
       <limit effort="0" lower="${-90*d2r}" upper="${90*d2r}" velocity="0"/>
@@ -142,5 +170,4 @@
     </joint>
     <link name="${namespace}/fin${fin_id}">
-      <!--<xacro:no_inertial/>-->
       <visual>
           <origin xyz="0 0 0" rpy="0 0 0"/>
@@ -173,13 +200,27 @@
           <joint_name>${namespace}/fin${fin_id}_joint</joint_name>
       </plugin>
-    </gazebo>
+    </gazebo>-->
   </xacro:macro>
   <xacro:property name="aft_fin_area" value="2.656049"/>
   <!--<xacro:property name="aft_fin_area" value="0.785"/>-->
-  <xacro:property name="aft_fin_lift_coefficient" value="19.1395"/>
-  <xacro:property name="aft_fin_drag_coefficient" value="1.98"/>
+  <xacro:property name="aft_fin_lift_coefficient" value="1.74975211"/>
+  <xacro:property name="aft_fin_drag_coefficient" value="0.269448395"/>
   <xacro:macro name="back_up_fin_macro" params="namespace fin_id *origin mesh_filename">
+    <xacro:lat_up_fin_quadratic_macro
+        namespace="${namespace}"
+        parent_link="${namespace}/base_link"
+        fin_id="${fin_id}"
+        min_joint_limit="${-90.0*d2r}"
+        max_joint_limit="${90.0*d2r}"
+        mesh_filename="${mesh_filename}"
+        fin_dynamics_time_constant="0.2"
+        lift_constant="${0.5 * fin_rho * aft_fin_area * aft_fin_lift_coefficient}"
+        drag_constant="${0.5 * fin_rho * aft_fin_area * aft_fin_drag_coefficient}"
+        current_velocity_topic="current_velocity">
+        <xacro:insert_block name="origin"/>
+    </xacro:lat_up_fin_quadratic_macro>
+    <!--<link name="${namespace}/fin${fin_id}">
+      <visual>
     <link name="${namespace}/fin${fin_id}">
-      <!--<xacro:no_inertial/>-->
       <visual>
           <origin xyz="0 0 0" rpy="0 0 0"/>
@@ -217,9 +258,23 @@
           <joint_name>${namespace}/fin${fin_id}_joint</joint_name>
       </plugin>
-    </gazebo>
+    </gazebo>-->
   </xacro:macro>
   <xacro:macro name="back_down_fin_macro" params="namespace fin_id *origin mesh_filename">
+    <xacro:lat_down_fin_quadratic_macro
+        namespace="${namespace}"
+        parent_link="${namespace}/base_link"
+        fin_id="${fin_id}"
+        min_joint_limit="${-90.0*d2r}"
+        max_joint_limit="${90.0*d2r}"
+        mesh_filename="${mesh_filename}"
+        fin_dynamics_time_constant="0.2"
+        lift_constant="${0.5 * fin_rho * aft_fin_area * aft_fin_lift_coefficient}"
+        drag_constant="${0.5 * fin_rho * aft_fin_area * aft_fin_drag_coefficient}"
+        current_velocity_topic="current_velocity">
+        <xacro:insert_block name="origin"/>
+    </xacro:lat_down_fin_quadratic_macro>
+    <!--<link name="${namespace}/fin${fin_id}">
+      <visual>
     <link name="${namespace}/fin${fin_id}">
-      <!--<xacro:no_inertial/>-->
       <visual>
           <origin xyz="0 0 0" rpy="0 0 0"/>
@@ -257,5 +312,5 @@
           <joint_name>${namespace}/fin${fin_id}_joint</joint_name>
       </plugin>
-    </gazebo>
+    </gazebo>-->
   </xacro:macro>
 </robot>
