Commit message: Update hydrodynamic model for 40m size model

File: urdf/actuators_original.xacro (robot description, xacro)
@@ -4,22 +4,22 @@
         <origin xyz="-21.77 0.0 0.0" rpy="0 0 0" />
     </xacro:thruster_macro>
-    <xacro:front_left_fin_macro namespace="${namespace}" fin_id="0" mesh_filename="${front_left_fin_mesh_file}">
-        <origin xyz="10.411 2.1937 1.20" rpy="0 0 0" />
-    </xacro:front_left_fin_macro>
-    <!--<xacro:front_right_fin_macro namespace="${namespace}" fin_id="1" mesh_filename="${front_left_fin_mesh_file}">-->
-    <xacro:front_right_fin_macro namespace="${namespace}" fin_id="1" mesh_filename="${front_right_fin_mesh_file}">
-        <origin xyz="10.411 -2.1937 1.20" rpy="0 0 0" />
-    </xacro:front_right_fin_macro>
-    <xacro:front_left_fin_macro namespace="${namespace}" fin_id="2" mesh_filename="${front_left_fin_mesh_file}">
-        <origin xyz="-16.385 2.0 0.395" rpy="0 0 0" />
-    </xacro:front_left_fin_macro>
-    <xacro:back_up_fin_macro namespace="${namespace}" fin_id="3" mesh_filename="${back_up_fin_mesh_file}">
+    <xacro:front_fin_macro namespace="${namespace}" fin_id="0" mesh_filename="${front_right_fin_mesh_file}">
+        <origin xyz="10.411 -2.1937 1.20" rpy="${-0.5 * pi}  0 0" />
+    </xacro:front_fin_macro>
+    <!--<xacro:front_fin_macro namespace="${namespace}" fin_id="1" mesh_filename="${front_left_fin_mesh_file}">-->
+    <xacro:front_fin_macro namespace="${namespace}" fin_id="1" mesh_filename="${front_left_fin_mesh_file}">
+        <origin xyz="10.411 2.1937 1.20" rpy="${-0.5 * pi} 0 0" />
+    </xacro:front_fin_macro>
+    <xacro:back_fin_macro namespace="${namespace}" fin_id="2" mesh_filename="${back_up_fin_mesh_file}">
+        <origin xyz="-16.385 -2.0 0.395" rpy="${0.5 * pi} 0 0" />
+    </xacro:back_fin_macro>
+    <xacro:back_fin_macro namespace="${namespace}" fin_id="3" mesh_filename="${back_up_fin_mesh_file}">
         <origin xyz="-16.385 0.0 1.8456" rpy="0 0 0"/>
-    </xacro:back_up_fin_macro>
-    <xacro:front_right_fin_macro namespace="${namespace}" fin_id="4" mesh_filename="${front_right_fin_mesh_file}">
-        <origin xyz="-16.385 -2.0 0.395" rpy="0 0 0" />
-    </xacro:front_right_fin_macro>
-    <xacro:back_down_fin_macro namespace="${namespace}" fin_id="5" mesh_filename="${back_down_fin_mesh_file}">
+    </xacro:back_fin_macro>
+    <xacro:back_fin_macro namespace="${namespace}" fin_id="4" mesh_filename="${back_down_fin_mesh_file}">
+        <origin xyz="-16.385 2.0 0.395" rpy="${0.5 * pi}  0 0" />
+    </xacro:back_fin_macro>
+    <xacro:back_fin_macro namespace="${namespace}" fin_id="5" mesh_filename="${back_down_fin_mesh_file}">
         <origin xyz="-16.385 0.0 -1.8456" rpy="0 0 0"/>
-    </xacro:back_down_fin_macro>
+    </xacro:back_fin_macro>
 </robot>

File: urdf/base_original.xacro (robot description, xacro)
@@ -24,6 +24,6 @@
               <origin rpy="0 0 0" xyz="0 0 0"/>
               <geometry>
-                  <!--<mesh filename="package://O_29qt/meshes/base_link_ano.STL" scale="1 1 1"/>-->
-                  <mesh filename="file://$(find O_29qt)/meshes/O_29_base.dae" scale="1 1 1"/>
+                  <!--<mesh filename="file://$(find O_29qt)/meshes/O_29_base.dae" scale="1 1 1"/>-->
+                  <mesh filename="file://$(find O_29qt)/meshes/40m/O_29base_40m.dae" scale="1 1 1"/>
               </geometry>
               <!--<material name="">
@@ -34,6 +34,6 @@
               <origin rpy="0 0 0" xyz="0 0 0"/>
               <geometry>
-                  <!--<mesh filename="package://O_29qt/meshes/base_link_ano.STL" scale="1 1 1"/>-->
-                  <mesh filename="file://$(find O_29qt)/meshes/O_29_base.dae" scale="1 1 1"/>
+                  <!--<mesh filename="file://$(find O_29qt)/meshes/O_29_base.dae" scale="1 1 1"/>-->
+                  <mesh filename="file://$(find O_29qt)/meshes/40m/O_29base_40m.dae" scale="1 1 1"/>
               </geometry>
             </collision>

File: urdf/gazebo_original.xacro (robot description, xacro)
@@ -10,7 +10,7 @@
     <!-- Describing the dimensions of the vehicle's bounding box -->
     <xacro:property name="O_29qt_length" value="40.97"/>
-    <xacro:property name="O_29qt_width"  value="4.923"/>
-    <xacro:property name="O_29qt_radius"  value="2.4615"/>
-    <xacro:property name="O_29qt_height" value="4.923"/>
+    <xacro:property name="O_29qt_width"  value="7.8894"/>
+    <xacro:property name="O_29qt_radius"  value="2.4616"/>
+    <xacro:property name="O_29qt_height" value="7.4994"/>
     <!-- Added base parameters(ARMSAUA) -->
     <!--<xacro:property name="O_29qt_length" value="2.712"/>
@@ -127,19 +127,11 @@
           <type>fossen</type>
           <added_mass>
-              ${-xudot*D3*0.1}      ${-xvdot*D3*0.1}       ${-xwdot*D3*0.1}       ${-xpdot*D4*0.1}      ${-xqdot*D4*0.1}      ${-xrdot*D4*0.1}
-              ${-yudot*D3*0.1}      ${-yvdot*D3*0.1}       ${-ywdot*D3*0.1}       ${-ypdot*D4*0.1}      ${-yqdot*D4*0.1}      ${-yrdot*D4*0.1}
-              ${-zudot*D3*0.1}      ${-zvdot*D3*0.1}       ${-zwdot*D3*0.1}       ${-zpdot*D4*0.1}      ${-zqdot*D4*0.1}      ${-zrdot*D4*0.1}
-              ${-kudot*D4*0.1}      ${-kvdot*D4*0.1}       ${-kwdot*D4*0.1}       ${-kpdot*D5*0.1}      ${-kqdot*D5*0.1}      ${-krdot*D5*0.1}
-              ${-mudot*D4*0.1}      ${-mvdot*D4*0.1}       ${-mwdot*D4*0.1}       ${-mpdot*D5*0.1}      ${-mqdot*D5*0.1}      ${-mrdot*D5*0.1}
-              ${-nudot*D4*0.1}      ${-nvdot*D4*0.1}       ${-nwdot*D4*0.1}       ${-npdot*D5*0.1}      ${-nqdot*D5*0.1}      ${-nrdot*D5*0.1}
+              ${xudot*D3*0.1}      ${xvdot*D3*0.1}       ${xwdot*D3*0.1}       ${xpdot*D4*0.1}      ${xqdot*D4*0.1}      ${xrdot*D4*0.1}
+              ${yudot*D3*0.1}      ${yvdot*D3*0.1}       ${ywdot*D3*0.1}       ${ypdot*D4*0.1}      ${yqdot*D4*0.1}      ${yrdot*D4*0.1}
+              ${zudot*D3*0.1}      ${zvdot*D3*0.1}       ${zwdot*D3*0.1}       ${zpdot*D4*0.1}      ${zqdot*D4*0.1}      ${zrdot*D4*0.1}
+              ${kudot*D4*0.1}      ${kvdot*D4*0.1}       ${kwdot*D4*0.1}       ${kpdot*D5*0.1}      ${kqdot*D5*0.1}      ${krdot*D5*0.1}
+              ${mudot*D4*0.1}      ${mvdot*D4*0.1}       ${mwdot*D4*0.1}       ${mpdot*D5*0.1}      ${mqdot*D5*0.1}      ${mrdot*D5*0.1}
+              ${nudot*D4*0.1}      ${nvdot*D4*0.1}       ${nwdot*D4*0.1}       ${npdot*D5*0.1}      ${nqdot*D5*0.1}      ${nrdot*D5*0.1}
           </added_mass>
-          <!--<added_mass>
-            1.432   0       0       0     0      0
-            0    120.645    0       0     0    4.895
-            0       0    130.513    0  -16.488   0
-            0       0       0    0.386    0      0
-            0       0   -16.488     0  78.266    0
-            0     4.895     0       0     0    67.489
-          </added_mass>-->
           <!--
             The linear damping coefficients can be provided as a diagonal (6 elements)

File: urdf/snippets_original.xacro (robot description, xacro)
@@ -39,7 +39,7 @@
                 <clampMin>-2500</clampMin>
                 <!-- Maximum thrust force output allowed -->
-                <thrustMax>263388.11</thrustMax>
+                <thrustMax>2633881.1</thrustMax>
                 <!-- Minimum thrust force output allowed -->
-                <thrustMin>-263388.11</thrustMin>
+                <thrustMin>-2633881.1</thrustMin>
                 <!--
                 Value from 0 to 1 to set the efficiency of the output thrus
@@ -75,5 +75,5 @@
                     <type>LinearInterp</type>
                     <inputValues>0 500 1000 1500 2000 2500</inputValues>
-                    <outputValues>0 10535.524 42142.097 94819.719 168568.39 263388.11</outputValues>
+                    <outputValues>0 105355.24 421420.97 948197.19 1685683.9 2633881.1</outputValues>
                 </conversion>
             </plugin>
@@ -85,8 +85,8 @@
     <!-- MACRO FOR FIN/RUDDER UNITS  -->
   <!-- A separate mesh for the fin should be stored in the meshes folder -->
-  <xacro:property name="front_left_fin_mesh_file" value="file://$(find O_29qt)/meshes/front_fin_left_new.dae"/>
-  <xacro:property name="front_right_fin_mesh_file" value="file://$(find O_29qt)/meshes/front_fin_right_new.dae"/>
-  <xacro:property name="back_up_fin_mesh_file" value="file://$(find O_29qt)/meshes/back_fin_up_new.dae"/>
-  <xacro:property name="back_down_fin_mesh_file" value="file://$(find O_29qt)/meshes/back_fin_down_new.dae"/>
+  <xacro:property name="front_left_fin_mesh_file" value="file://$(find O_29qt)/meshes/40m/front_left_fin_40m.dae"/>
+  <xacro:property name="front_right_fin_mesh_file" value="file://$(find O_29qt)/meshes/40m/front_right_fin_40m.dae"/>
+  <xacro:property name="back_up_fin_mesh_file" value="file://$(find O_29qt)/meshes/40m/back_up_fin_40m.dae"/>
+  <xacro:property name="back_down_fin_mesh_file" value="file://$(find O_29qt)/meshes/40m/back_down_fin_40m.dae"/>
   <!-- Fin properties -->
   <xacro:property name="fin_rho" value="1025"/>
@@ -94,11 +94,14 @@
   <xacro:property name="front_fin_lift_coefficient" value="1.668475641"/>
   <xacro:property name="front_fin_drag_coefficient" value="0.26542681"/>
-  <xacro:macro name="front_left_fin_macro" params="namespace fin_id *origin mesh_filename">
-    <xacro:hor_left_fin_quadratic_macro
+  <xacro:property name="back_fin_area" value="2.656049"/>
+  <xacro:property name="back_fin_lift_coefficient" value="1.74975211"/>
+  <xacro:property name="back_fin_drag_coefficient" value="0.269448395"/>
+  <xacro:macro name="front_fin_macro" params="namespace fin_id *origin mesh_filename">
+      <xacro:fin_quadratic_macro
         namespace="${namespace}"
         parent_link="${namespace}/base_link"
         fin_id="${fin_id}"
-        min_joint_limit="${-90.0*d2r}"
-        max_joint_limit="${90.0*d2r}"
+        min_joint_limit="${-90.0 * d2r}"
+        max_joint_limit="${90.0 * d2r}"
         mesh_filename="${mesh_filename}"
         fin_dynamics_time_constant="0.2"
@@ -107,210 +110,20 @@
         current_velocity_topic="current_velocity">
         <xacro:insert_block name="origin"/>
-    </xacro:hor_left_fin_quadratic_macro>
-    <!--<link name="${namespace}/fin${fin_id}">
-      <visual>
-          <origin xyz="0 0 0" rpy="0 0 0"/>
-          <geometry>
-              <mesh filename="${mesh_filename}" scale="1 1 1"/>
-          </geometry>
-      </visual>
-      <inertial>
-          <mass value="0.001" />
-          <origin xyz="0 0 0" rpy="0 0 0" />
-          <inertia ixx="0.000000001" ixy="0.0" ixz="0.0" iyy="0.000000001" iyz="0.0" izz="0.000000001" />
-      </inertial>
-    </link>
-    <joint name="${namespace}/fin${fin_id}_joint" type="revolute">
-      <limit effort="0" lower="${-90*d2r}" upper="${90*d2r}" velocity="0"/>
-      <xacro:insert_block name="origin"/>
-      <xacro:insert_block name="axiz"/>
-      <parent link="${namespace}/base_link"/>
-      <child link="${namespace}/fin${fin_id}"/>
-    </joint>
-    <gazebo>
-      <plugin name="${namespace}_fin${fin_id}_model" filename="libuuv_fin_ros_plugin.so">
-          <dynamics>
-              <type>FirstOrder</type>
-              <timeConstant>0.2</timeConstant>
-          </dynamics>
-          <liftdrag>
-              <type>Quadratic</type>
-              <lift_constant>${0.5 * fin_rho * front_fin_area * front_fin_lift_coefficient}</lift_constant>
-              <drag_constant>${0.5 * fin_rho * front_fin_area * front_fin_drag_coefficient}</drag_constant>
-          </liftdrag>
-          <current_velocity_topic>current_velocity</current_velocity_topic>
-          <fin_id>${fin_id}</fin_id>
-          <link_name>${namespace}/fin${fin_id}</link_name>
-          <joint_name>${namespace}/fin${fin_id}_joint</joint_name>
-      </plugin>
-    </gazebo>-->
+      </xacro:fin_quadratic_macro>
   </xacro:macro>
-  <xacro:macro name="front_right_fin_macro" params="namespace fin_id *origin mesh_filename">
-    <xacro:hor_right_fin_quadratic_macro
+  <xacro:macro name="back_fin_macro" params="namespace fin_id *origin mesh_filename">
+      <xacro:fin_quadratic_macro
         namespace="${namespace}"
         parent_link="${namespace}/base_link"
         fin_id="${fin_id}"
-        min_joint_limit="${-90.0*d2r}"
-        max_joint_limit="${90.0*d2r}"
+        min_joint_limit="${-90.0 * d2r}"
+        max_joint_limit="${90.0 * d2r}"
         mesh_filename="${mesh_filename}"
         fin_dynamics_time_constant="0.2"
-        lift_constant="${0.5 * fin_rho * front_fin_area * front_fin_lift_coefficient}"
-        drag_constant="${0.5 * fin_rho * front_fin_area * front_fin_drag_coefficient}"
+        lift_constant="${0.5 * fin_rho * back_fin_area * back_fin_lift_coefficient}"
+        drag_constant="${0.5 * fin_rho * back_fin_area * back_fin_drag_coefficient}"
         current_velocity_topic="current_velocity">
         <xacro:insert_block name="origin"/>
-    </xacro:hor_right_fin_quadratic_macro>
-    <!--<link name="${namespace}/fin${fin_id}">
-      <visual>
-    <joint name="${namespace}/fin${fin_id}_joint" type="revolute">
-      <limit effort="0" lower="${-90*d2r}" upper="${90*d2r}" velocity="0"/>
-      <xacro:insert_block name="origin"/>
-      <xacro:insert_block name="axiz"/>
-      <parent link="${namespace}/base_link"/>
-      <child link="${namespace}/fin${fin_id}"/>
-    </joint>
-    <link name="${namespace}/fin${fin_id}">
-      <visual>
-          <origin xyz="0 0 0" rpy="0 0 0"/>
-          <geometry>
-              <mesh filename="${mesh_filename}" scale="1 -1 1"/>
-          </geometry>
-      </visual>
-      <inertial>
-          <mass value="0.001" />
-          <origin xyz="0 0 0" rpy="0 0 0" />
-          <inertia ixx="0.000000001" ixy="0.0" ixz="0.0"
-              iyy="0.000000001" iyz="0.0"
-              izz="0.000000001" />
-      </inertial>
-    </link>
-    <gazebo>
-      <plugin name="${namespace}_fin${fin_id}_model" filename="libuuv_fin_ros_plugin.so">
-          <dynamics>
-              <type>FirstOrder</type>
-              <timeConstant>0.2</timeConstant>
-          </dynamics>
-          <liftdrag>
-              <type>Quadratic</type>
-              <lift_constant>${0.5 * fin_rho * front_fin_area * front_fin_lift_coefficient}</lift_constant>
-              <drag_constant>${0.5 * fin_rho * front_fin_area * front_fin_drag_coefficient}</drag_constant>
-          </liftdrag>
-          <current_velocity_topic>current_velocity</current_velocity_topic>
-          <fin_id>${fin_id}</fin_id>
-          <link_name>${namespace}/fin${fin_id}</link_name>
-          <joint_name>${namespace}/fin${fin_id}_joint</joint_name>
-      </plugin>
-    </gazebo>-->
-  </xacro:macro>
-  <xacro:property name="aft_fin_area" value="2.656049"/>
-  <!--<xacro:property name="aft_fin_area" value="0.785"/>-->
-  <xacro:property name="aft_fin_lift_coefficient" value="1.74975211"/>
-  <xacro:property name="aft_fin_drag_coefficient" value="0.269448395"/>
-  <xacro:macro name="back_up_fin_macro" params="namespace fin_id *origin mesh_filename">
-    <xacro:lat_up_fin_quadratic_macro
-        namespace="${namespace}"
-        parent_link="${namespace}/base_link"
-        fin_id="${fin_id}"
-        min_joint_limit="${-90.0*d2r}"
-        max_joint_limit="${90.0*d2r}"
-        mesh_filename="${mesh_filename}"
-        fin_dynamics_time_constant="0.2"
-        lift_constant="${0.5 * fin_rho * aft_fin_area * aft_fin_lift_coefficient}"
-        drag_constant="${0.5 * fin_rho * aft_fin_area * aft_fin_drag_coefficient}"
-        current_velocity_topic="current_velocity">
-        <xacro:insert_block name="origin"/>
-    </xacro:lat_up_fin_quadratic_macro>
-    <!--<link name="${namespace}/fin${fin_id}">
-      <visual>
-    <link name="${namespace}/fin${fin_id}">
-      <visual>
-          <origin xyz="0 0 0" rpy="0 0 0"/>
-          <geometry>
-              <mesh filename="${mesh_filename}" scale="1 1 1"/>
-          </geometry>
-      </visual>
-      <inertial>
-          <mass value="0.001" />
-          <origin xyz="0 0 0" rpy="0 0 0" />
-          <inertia ixx="0.000000001" ixy="0.0" ixz="0.0" iyy="0.000000001" iyz="0.0" izz="0.000000001" />
-      </inertial>
-    </link>
-    <joint name="${namespace}/fin${fin_id}_joint" type="revolute">
-      <limit effort="0" lower="${-90*d2r}" upper="${90*d2r}" velocity="0"/>
-      <xacro:insert_block name="origin"/>
-      <axiz xyz="0 0 1"/>
-      <parent link="${namespace}/base_link"/>
-      <child link="${namespace}/fin${fin_id}"/>
-    </joint>
-    <gazebo>
-      <plugin name="${namespace}_fin${fin_id}_model" filename="libuuv_fin_ros_plugin.so">
-          <dynamics>
-              <type>FirstOrder</type>
-              <timeConstant>0.2</timeConstant>
-          </dynamics>
-          <liftdrag>
-              <type>Quadratic</type>
-              <lift_constant>${0.5 * fin_rho * aft_fin_area * aft_fin_lift_coefficient}</lift_constant>
-              <drag_constant>${0.5 * fin_rho * aft_fin_area * aft_fin_drag_coefficient}</drag_constant>
-          </liftdrag>
-          <current_velocity_topic>current_velocity</current_velocity_topic>
-          <fin_id>${fin_id}</fin_id>
-          <link_name>${namespace}/fin${fin_id}</link_name>
-          <joint_name>${namespace}/fin${fin_id}_joint</joint_name>
-      </plugin>
-    </gazebo>-->
-  </xacro:macro>
-  <xacro:macro name="back_down_fin_macro" params="namespace fin_id *origin mesh_filename">
-    <xacro:lat_down_fin_quadratic_macro
-        namespace="${namespace}"
-        parent_link="${namespace}/base_link"
-        fin_id="${fin_id}"
-        min_joint_limit="${-90.0*d2r}"
-        max_joint_limit="${90.0*d2r}"
-        mesh_filename="${mesh_filename}"
-        fin_dynamics_time_constant="0.2"
-        lift_constant="${0.5 * fin_rho * aft_fin_area * aft_fin_lift_coefficient}"
-        drag_constant="${0.5 * fin_rho * aft_fin_area * aft_fin_drag_coefficient}"
-        current_velocity_topic="current_velocity">
-        <xacro:insert_block name="origin"/>
-    </xacro:lat_down_fin_quadratic_macro>
-    <!--<link name="${namespace}/fin${fin_id}">
-      <visual>
-    <link name="${namespace}/fin${fin_id}">
-      <visual>
-          <origin xyz="0 0 0" rpy="0 0 0"/>
-          <geometry>
-              <mesh filename="${mesh_filename}" scale="1 1 -1"/>
-          </geometry>
-      </visual>
-      <inertial>
-          <mass value="0.001" />
-          <origin xyz="0 0 0" rpy="0 0 0" />
-          <inertia ixx="0.000000001" ixy="0.0" ixz="0.0" iyy="0.000000001" iyz="0.0" izz="0.000000001" />
-      </inertial>
-    </link>
-    <joint name="${namespace}/fin${fin_id}_joint" type="revolute">
-      <limit effort="0" lower="${-90*d2r}" upper="${90*d2r}" velocity="0"/>
-      <xacro:insert_block name="origin"/>
-      <axiz xyz="0 0 1"/>
-      <parent link="${namespace}/base_link"/>
-      <child link="${namespace}/fin${fin_id}"/>
-    </joint>
-    <gazebo>
-      <plugin name="${namespace}_fin${fin_id}_model" filename="libuuv_fin_ros_plugin.so">
-          <dynamics>
-              <type>FirstOrder</type>
-              <timeConstant>0.2</timeConstant>
-          </dynamics>
-          <liftdrag>
-              <type>Quadratic</type>
-              <lift_constant>${0.5 * fin_rho * aft_fin_area * aft_fin_lift_coefficient}</lift_constant>
-              <drag_constant>${0.5 * fin_rho * aft_fin_area * aft_fin_drag_coefficient}</drag_constant>
-          </liftdrag>
-          <current_velocity_topic>current_velocity</current_velocity_topic>
-          <fin_id>${fin_id}</fin_id>
-          <link_name>${namespace}/fin${fin_id}</link_name>
-          <joint_name>${namespace}/fin${fin_id}_joint</joint_name>
-      </plugin>
-    </gazebo>-->
+      </xacro:fin_quadratic_macro>
   </xacro:macro>
 </robot>
